File: PCB/PCB.sch (KiCad schematic (older format))
At the start: 2 parts

Commit message: footprint update
Parts:
- added J?: USB_B, Connector_USB:USB_B_OST_USB-B1HSxx_Horizontal, symbol Connector:USB_B
Connections:
- net GND: now reaches U?.1 (GND)
- net GND: now also J?.4 (GND)
- net at U?.5 (UD+): now also J?.3 (D+)
- net at U?.6 (UD-): now also J?.2 (D-)
Changed lines of the file:
@@
 EESchema Schematic File Version 4
+LIBS:PCB-cache
 EELAYER 30 0
 EELAYER END
@@
 L Interface_USB:CH340G U?
 U 1 1 5D6724AA
-P 8100 2150
-F 0 "U?" H 8100 1461 50  0000 C CNN
-F 1 "CH340G" H 8100 1370 50  0000 C CNN
-F 2 "Package_SO:SOIC-16_3.9x9.9mm_P1.27mm" H 8150 1600 50  0001 L CNN
-F 3 "http://www.datasheet5.com/pdf-local-2195953" H 7750 2950 50  0001 C CNN
-	1    8100 2150
+P 8500 1800
+F 0 "U?" H 8500 1111 50  0001 C CNN
+F 1 "CH340G" H 8500 1020 50  0000 C CNN
+F 2 "Package_SO:SOIC-16_3.9x9.9mm_P1.27mm" H 8550 1250 50  0001 L CNN
+F 3 "http://www.datasheet5.com/pdf-local-2195953" H 8150 2600 50  0001 C CNN
+	1    8500 1800
+	-1   0    0    1
+$EndComp
+$Comp
+L Connector:USB_B J?
+U 1 1 5D670289
+P 9700 1900
+F 0 "J?" H 9470 1797 50  0001 R CNN
+F 1 "USB_B" H 9470 1843 50  0000 R CNN
+F 2 "Connector_USB:USB_B_OST_USB-B1HSxx_Horizontal" H 9850 1850 50  0001 C CNN
+F 3 " ~" H 9850 1850 50  0001 C CNN
+	1    9700 1900
+	-1   0    0    1
+$EndComp
+$Comp
+L power:GND #PWR?
+U 1 1 5D677A17
+P 9450 1350
+F 0 "#PWR?" H 9450 1100 50  0001 C CNN
+F 1 "GND" H 9455 1177 50  0000 C CNN
+F 2 "" H 9450 1350 50  0001 C CNN
+F 3 "" H 9450 1350 50  0001 C CNN
+	1    9450 1350
 	1    0    0    -1
 $EndComp
+$Comp
+L power:GND #PWR?
+U 1 1 5D677FB5
+P 8700 1050
+F 0 "#PWR?" H 8700 800 50  0001 C CNN
+F 1 "GND" H 8705 877 50  0000 C CNN
+F 2 "" H 8700 1050 50  0001 C CNN
+F 3 "" H 8700 1050 50  0001 C CNN
+	1    8700 1050
+	1    0    0    -1
+$EndComp
+Wire Wire Line
+	9700 1500 9700 1200
+Wire Wire Line
+	9700 1200 9450 1200
+Wire Wire Line
+	9450 1200 9450 1350
+Wire Wire Line
+	8700 1050 8700 900
+Wire Wire Line
+	8700 900  8500 900
+Wire Wire Line
+	8500 900  8500 1200
+Wire Wire Line
+	8900 1800 9400 1800
+Wire Wire Line
+	9400 1900 8900 1900
 $EndSCHEMATC

Commit message: uprava PCB
Connections:
- net GND: now also U?.1 (GND), U?.15 (GND), U?.38 (GND)
Changed lines of the file:
@@
 EESchema Schematic File Version 4
-LIBS:PCB-cache
 EELAYER 30 0
 EELAYER END
@@
 L Interface_USB:CH340G U?
 U 1 1 5D6724AA
-P 8500 1800
-F 0 "U?" H 8500 1111 50  0001 C CNN
-F 1 "CH340G" H 8500 1020 50  0000 C CNN
-F 2 "Package_SO:SOIC-16_3.9x9.9mm_P1.27mm" H 8550 1250 50  0001 L CNN
-F 3 "http://www.datasheet5.com/pdf-local-2195953" H 8150 2600 50  0001 C CNN
-	1    8500 1800
-	-1   0    0    1
+P 2300 1750
+F 0 "U?" H 2300 1061 50  0001 C CNN
+F 1 "CH340G" H 2300 970 50  0000 C CNN
+F 2 "Package_SO:SOIC-16_3.9x9.9mm_P1.27mm" H 2350 1200 50  0001 L CNN
+F 3 "http://www.datasheet5.com/pdf-local-2195953" H 1950 2550 50  0001 C CNN
+	1    2300 1750
+	1    0    0    -1
 $EndComp
 $Comp
 L Connector:USB_B J?
 U 1 1 5D670289
-P 9700 1900
-F 0 "J?" H 9470 1797 50  0001 R CNN
-F 1 "USB_B" H 9470 1843 50  0000 R CNN
-F 2 "Connector_USB:USB_B_OST_USB-B1HSxx_Horizontal" H 9850 1850 50  0001 C CNN
-F 3 " ~" H 9850 1850 50  0001 C CNN
-	1    9700 1900
-	-1   0    0    1
+P 1100 1650
+F 0 "J?" H 870 1547 50  0001 R CNN
+F 1 "USB_B" H 870 1593 50  0000 R CNN
+F 2 "Connector_USB:USB_B_OST_USB-B1HSxx_Horizontal" H 1250 1600 50  0001 C CNN
+F 3 " ~" H 1250 1600 50  0001 C CNN
+	1    1100 1650
+	1    0    0    -1
 $EndComp
+Wire Wire Line
+	1900 1750 1400 1750
+Wire Wire Line
+	1400 1650 1900 1650
 $Comp
 L power:GND #PWR?
-U 1 1 5D677A17
-P 9450 1350
-F 0 "#PWR?" H 9450 1100 50  0001 C CNN
-F 1 "GND" H 9455 1177 50  0000 C CNN
-F 2 "" H 9450 1350 50  0001 C CNN
-F 3 "" H 9450 1350 50  0001 C CNN
-	1    9450 1350
+U 1 1 5D69F6EE
+P 1100 2350
+F 0 "#PWR?" H 1100 2100 50  0001 C CNN
+F 1 "GND" H 1105 2177 50  0000 C CNN
+F 2 "" H 1100 2350 50  0001 C CNN
+F 3 "" H 1100 2350 50  0001 C CNN
+	1    1100 2350
 	1    0    0    -1
 $EndComp
 $Comp
 L power:GND #PWR?
-U 1 1 5D677FB5
-P 8700 1050
-F 0 "#PWR?" H 8700 800 50  0001 C CNN
-F 1 "GND" H 8705 877 50  0000 C CNN
-F 2 "" H 8700 1050 50  0001 C CNN
-F 3 "" H 8700 1050 50  0001 C CNN
-	1    8700 1050
+U 1 1 5D69F9AA
+P 2300 2650
+F 0 "#PWR?" H 2300 2400 50  0001 C CNN
+F 1 "GND" H 2305 2477 50  0000 C CNN
+F 2 "" H 2300 2650 50  0001 C CNN
+F 3 "" H 2300 2650 50  0001 C CNN
+	1    2300 2650
 	1    0    0    -1
 $EndComp
 Wire Wire Line
-	9700 1500 9700 1200
+	2300 2350 2300 2650
 Wire Wire Line
-	9700 1200 9450 1200
+	1100 2050 1100 2350
+$Comp
+L power:GND #PWR?
+U 1 1 5D6A10B5
+P 4300 5450
+F 0 "#PWR?" H 4300 5200 50  0001 C CNN
+F 1 "GND" H 4305 5277 50  0000 C CNN
+F 2 "" H 4300 5450 50  0001 C CNN
+F 3 "" H 4300 5450 50  0001 C CNN
+	1    4300 5450
+	1    0    0    -1
+$EndComp
 Wire Wire Line
-	9450 1200 9450 1350
-Wire Wire Line
-	8700 1050 8700 900
-Wire Wire Line
-	8700 900  8500 900
-Wire Wire Line
-	8500 900  8500 1200
-Wire Wire Line
-	8900 1800 9400 1800
-Wire Wire Line
-	9400 1900 8900 1900
+	4300 5200 4300 5450
 $EndSCHEMATC

Commit message: pcb modified
Parts:
- added C?: 0.1uF, Capacitor_THT:C_Disc_D3.0mm_W2.0mm_P2.50mm, symbol Device:C
- added C?: 2.2uF, symbol Device:CP
- added C?: 100nF, symbol Device:C
- added POWER: 12V, Connector_PinHeader_2.54mm:PinHeader_1x03_P2.54mm_Horizontal, symbol Connector_Generic:Conn_01x03
- added U?: LF33_TO220, Package_TO_SOT_THT:TO-220-3_Vertical, symbol Regulator_Linear:LF33_TO220
Connections:
- wire segments 5 -> 33
Other:
- moved on the sheet: U?
Changed lines of the file:
@@
 EESchema Schematic File Version 4
+LIBS:PCB-cache
 EELAYER 30 0
 EELAYER END
@@
 L RF_Module:ESP32-WROOM-32 U?
 U 1 1 5D66FD00
-P 4300 3800
-F 0 "U?" H 4300 5381 50  0000 C CNN
-F 1 "ESP32-WROOM-32" H 4300 5290 50  0000 C CNN
-F 2 "RF_Module:ESP32-WROOM-32" H 4300 2300 50  0001 C CNN
-F 3 "https://www.espressif.com/sites/default/files/documentation/esp32-wroom-32_datasheet_en.pdf" H 4000 3850 50  0001 C CNN
-	1    4300 3800
-	1    0    0    -1
+P 4850 3550
+F 0 "U?" H 4850 5131 50  0000 C CNN
+F 1 "ESP32-WROOM-32" H 4850 5040 50  0000 C CNN
+F 2 "RF_Module:ESP32-WROOM-32" H 4850 2050 50  0001 C CNN
+F 3 "https://www.espressif.com/sites/default/files/documentation/esp32-wroom-32_datasheet_en.pdf" H 4550 3600 50  0001 C CNN
+	1    4850 3550
+	0    -1   -1   0
 $EndComp
 $Comp
@@
 $Comp
 L power:GND #PWR?
-U 1 1 5D6A10B5
-P 4300 5450
-F 0 "#PWR?" H 4300 5200 50  0001 C CNN
-F 1 "GND" H 4305 5277 50  0000 C CNN
-F 2 "" H 4300 5450 50  0001 C CNN
-F 3 "" H 4300 5450 50  0001 C CNN
-	1    4300 5450
-	1    0    0    -1
-$EndComp
-Wire Wire Line
-	4300 5200 4300 5450
+U 1 1 5D6DECAD
+P 6400 3700
+F 0 "#PWR?" H 6400 3450 50  0001 C CNN
+F 1 "GND" H 6405 3527 50  0000 C CNN
+F 2 "" H 6400 3700 50  0001 C CNN
+F 3 "" H 6400 3700 50  0001 C CNN
+	1    6400 3700
+	1    0    0    -1
+$EndComp
+Wire Wire Line
+	6250 3550 6400 3550
+Wire Wire Line
+	6400 3550 6400 3700
+Wire Wire Line
+	2700 1450 3750 1450
+Wire Wire Line
+	3750 1450 3750 2950
+Wire Wire Line
+	2700 1350 3950 1350
+Wire Wire Line
+	3950 1350 3950 2950
+$Comp
+L Connector_Generic:Conn_01x03 POWER
+U 1 1 5D6F0708
+P 750 3050
+F 0 "POWER" H 668 2725 50  0000 C CNN
+F 1 "12V" H 668 2816 50  0000 C CNN
+F 2 "Connector_PinHeader_2.54mm:PinHeader_1x03_P2.54mm_Horizontal" H 750 3050 50  0001 C CNN
+F 3 "~" H 750 3050 50  0001 C CNN
+	1    750  3050
+	-1   0    0    1
+$EndComp
+$Comp
+L power:GND #PWR?
+U 1 1 5D6F133A
+P 1100 3350
+F 0 "#PWR?" H 1100 3100 50  0001 C CNN
+F 1 "GND" H 1105 3177 50  0000 C CNN
+F 2 "" H 1100 3350 50  0001 C CNN
+F 3 "" H 1100 3350 50  0001 C CNN
+	1    1100 3350
+	1    0    0    -1
+$EndComp
+Wire Wire Line
+	950  3150 1100 3150
+Wire Wire Line
+	1100 3150 1100 3350
+Wire Wire Line
+	950  2950 1100 2950
+Wire Wire Line
+	1100 2950 1100 3150
+Connection ~ 1100 3150
+Wire Wire Line
+	2300 950  2300 1150
+$Comp
+L Device:C C?
+U 1 1 5D6F6BC7
+P 2600 950
+F 0 "C?" V 2348 950 50  0001 C CNN
+F 1 "0.1uF" V 2440 950 50  0000 C CNN
+F 2 "Capacitor_THT:C_Disc_D3.0mm_W2.0mm_P2.50mm" H 2638 800 50  0001 C CNN
+F 3 "~" H 2600 950 50  0001 C CNN
+	1    2600 950
+	0    1    1    0
+$EndComp
+$Comp
+L power:GND #PWR?
+U 1 1 5D6F78B6
+P 2850 1050
+F 0 "#PWR?" H 2850 800 50  0001 C CNN
+F 1 "GND" H 2855 877 50  0000 C CNN
+F 2 "" H 2850 1050 50  0001 C CNN
+F 3 "" H 2850 1050 50  0001 C CNN
+	1    2850 1050
+	1    0    0    -1
+$EndComp
+Wire Wire Line
+	2450 950  2300 950
+Wire Wire Line
+	2750 950  2850 950
+Wire Wire Line
+	2850 950  2850 1050
+$Comp
+L Regulator_Linear:LF33_TO220 U?
+U 1 1 5D6FD6AD
+P 1750 2900
+F 0 "U?" H 1750 3142 50  0001 C CNN
+F 1 "LF33_TO220" H 1750 3051 50  0000 C CNN
+F 2 "Package_TO_SOT_THT:TO-220-3_Vertical" H 1750 3125 50  0001 C CIN
+F 3 "http://www.st.com/content/ccc/resource/technical/document/datasheet/c4/0e/7e/2a/be/bc/4c/bd/CD00000546.pdf/files/CD00000546.pdf/jcr:content/translations/en.CD00000546.pdf" H 1750 2850 50  0001 C CNN
+	1    1750 2900
+	1    0    0    -1
+$EndComp
+$Comp
+L Device:CP C?
+U 1 1 5D700DCC
+P 2150 3250
+F 0 "C?" H 2268 3296 50  0001 L CNN
+F 1 "2.2uF" H 2268 3250 50  0000 L CNN
+F 2 "" H 2188 3100 50  0001 C CNN
+F 3 "~" H 2150 3250 50  0001 C CNN
+	1    2150 3250
+	1    0    0    -1
+$EndComp
+$Comp
+L Device:C C?
+U 1 1 5D701A35
+P 1350 3250
+F 0 "C?" H 1465 3296 50  0001 L CNN
+F 1 "100nF" H 1465 3250 50  0000 L CNN
+F 2 "" H 1388 3100 50  0001 C CNN
+F 3 "~" H 1350 3250 50  0001 C CNN
+	1    1350 3250
+	1    0    0    -1
+$EndComp
+$Comp
+L power:GND #PWR?
+U 1 1 5D704172
+P 1350 3600
+F 0 "#PWR?" H 1350 3350 50  0001 C CNN
+F 1 "GND" H 1355 3427 50  0000 C CNN
+F 2 "" H 1350 3600 50  0001 C CNN
+F 3 "" H 1350 3600 50  0001 C CNN
+	1    1350 3600
+	1    0    0    -1
+$EndComp
+$Comp
+L power:GND #PWR?
+U 1 1 5D704519
+P 1750 3600
+F 0 "#PWR?" H 1750 3350 50  0001 C CNN
+F 1 "GND" H 1755 3427 50  0000 C CNN
+F 2 "" H 1750 3600 50  0001 C CNN
+F 3 "" H 1750 3600 50  0001 C CNN
+	1    1750 3600
+	1    0    0    -1
+$EndComp
+$Comp
+L power:GND #PWR?
+U 1 1 5D70475E
+P 2150 3600
+F 0 "#PWR?" H 2150 3350 50  0001 C CNN
+F 1 "GND" H 2155 3427 50  0000 C CNN
+F 2 "" H 2150 3600 50  0001 C CNN
+F 3 "" H 2150 3600 50  0001 C CNN
+	1    2150 3600
+	1    0    0    -1
+$EndComp
+Wire Wire Line
+	950  3050 1350 3050
+Wire Wire Line
+	1350 3050 1350 2900
+Wire Wire Line
+	1350 2900 1450 2900
+Wire Wire Line
+	1350 3100 1350 3050
+Connection ~ 1350 3050
+Wire Wire Line
+	1350 3400 1350 3600
+Wire Wire Line
+	1750 3200 1750 3600
+Wire Wire Line
+	2050 2900 2150 2900
+Wire Wire Line
+	2150 2900 2150 3100
+Wire Wire Line
+	2150 3400 2150 3600
+Wire Wire Line
+	2300 950  2200 950
+Wire Wire Line
+	1700 950  1700 2600
+Wire Wire Line
+	1700 2600 2150 2600
+Wire Wire Line
+	2150 2600 2150 2900
+Connection ~ 2300 950
+Connection ~ 2150 2900
+Connection ~ 2200 950
+Wire Wire Line
+	2200 950  1700 950
+Wire Wire Line
+	2200 950  2200 1150
 $EndSCHEMATC

Commit message: PCB update
Parts:
- removed C?: 0.1uF, Capacitor_THT:C_Disc_D3.0mm_W2.0mm_P2.50mm, symbol Device:C
- removed C?: 2.2uF, symbol Device:CP
- removed C?: 100nF, symbol Device:C
- removed J?: USB_B, Connector_USB:USB_B_OST_USB-B1HSxx_Horizontal, symbol Connector:USB_B
- removed POWER: 12V, Connector_PinHeader_2.54mm:PinHeader_1x03_P2.54mm_Horizontal, symbol Connector_Generic:Conn_01x03
- removed U?: ESP32-WROOM-32, RF_Module:ESP32-WROOM-32, symbol RF_Module:ESP32-WROOM-32
- removed U?: CH340G, Package_SO:SOIC-16_3.9x9.9mm_P1.27mm, symbol Interface_USB:CH340G
- removed U?: LF33_TO220, Package_TO_SOT_THT:TO-220-3_Vertical, symbol Regulator_Linear:LF33_TO220
- added C? (x2): 22pF, Capacitor_SMD:C_1206_3216Metric, symbol Device:C
- added C?: 0.1uF, Capacitor_SMD:C_1206_3216Metric, symbol Device:C
- added C?: 2.2uF, Capacitor_THT:CP_Radial_D5.0mm_P2.00mm, symbol Device:CP
- added J?: USB_B, Connector_USB:USB_B_OST_USB-B1HSxx_Horizontal, symbol Connector:USB_B
- added J?: power 12V, Connector_PinHeader_2.54mm:PinHeader_1x03_P2.54mm_Horizontal, symbol Connector_Generic:Conn_01x03
- added U?: CH340G, Package_SO:SOP-16_4.4x10.4mm_P1.27mm, symbol Interface_USB:CH340G
- added U?: LF33CDT, Package_TO_SOT_SMD:TO-252-2, symbol Regulator_Linear:LF33_TO220
- added Y?: 12MHz, Crystal:Crystal_HC49-U_Vertical, symbol Device:Crystal
Connections:
- wire segments 33 -> 38

Commit message: PCB update
Parts:
- added C5: 0.33uC, Capacitor_SMD:C_1206_3216Metric, symbol Device:C
- added C6: 0.1uC, Capacitor_SMD:C_1206_3216Metric, symbol Device:C
- added J3: DS18B20, Connector_PinHeader_2.54mm:PinHeader_1x02_P2.54mm_Horizontal, symbol Connector_Generic:Conn_01x02
- added J4: NEXTION 2.8\", Connector_PinHeader_2.54mm:PinHeader_1x04_P2.54mm_Horizontal, symbol Connector_Generic:Conn_01x04
- added R1: 4K7, Resistor_THT:R_Axial_DIN0207_L6.3mm_D2.5mm_P10.16mm_Horizontal, symbol Device:R
- added R2: 1k, Resistor_THT:R_Axial_DIN0207_L6.3mm_D2.5mm_P10.16mm_Horizontal, symbol Device:R
- added R3: 2k, Resistor_THT:R_Axial_DIN0207_L6.3mm_D2.5mm_P10.16mm_Horizontal, symbol Device:R
- added U2: ESP32-WROOM-32, RF_Module:ESP32-WROOM-32, symbol RF_Module:ESP32-WROOM-32
- added U4: L7805, Package_TO_SOT_SMD:TO-252-2, symbol Regulator_Linear:L7805
- gave numbers to parts that had none: 9
Connections:
- wire segments 38 -> 87

Commit message: PCB update
Parts:
- removed J3: DS18B20, Connector_PinHeader_2.54mm:PinHeader_1x02_P2.54mm_Horizontal, symbol Connector_Generic:Conn_01x02
- removed R1: 4K7, Resistor_THT:R_Axial_DIN0207_L6.3mm_D2.5mm_P10.16mm_Horizontal, symbol Device:R
- added J?: DS18B20, symbol Connector_Generic:Conn_01x03
- added J? (x3): 4pin FAN, Connector:FanPinHeader_1x04_P2.54mm_Vertical, symbol Connector_Generic:Conn_01x04
Connections:
- wire segments 87 -> 108
Changed lines of the file:
@@
 EESchema Schematic File Version 4
-LIBS:PCB-cache
 EELAYER 30 0
 EELAYER END
@@
 	4750 2000 4750 2850
 Wire Wire Line
-	4750 2850 4650 2850
-Wire Wire Line
 	4400 2100 4400 2000
 Connection ~ 4400 2000
@@
 $EndComp
 $Comp
-L Connector_Generic:Conn_01x02 J3
-U 1 1 5D71EC3A
-P 4100 3200
-F 0 "J3" H 4018 2875 50  0001 C CNN
-F 1 "DS18B20" H 4018 2967 50  0000 C CNN
-F 2 "Connector_PinHeader_2.54mm:PinHeader_1x02_P2.54mm_Horizontal" H 4100 3200 50  0001 C CNN
-F 3 "~" H 4100 3200 50  0001 C CNN
-	1    4100 3200
-	-1   0    0    1
-$EndComp
-$Comp
-L power:GND #PWR0107
-U 1 1 5D721FD8
-P 4300 3250
-F 0 "#PWR0107" H 4300 3000 50  0001 C CNN
-F 1 "GND" H 4305 3077 50  0000 C CNN
-F 2 "" H 4300 3250 50  0001 C CNN
-F 3 "" H 4300 3250 50  0001 C CNN
-	1    4300 3250
-	1    0    0    -1
-$EndComp
-Wire Wire Line
-	4300 3200 4300 3250
-Wire Wire Line
-	4500 3100 4300 3100
-$Comp
-L Device:R R1
-U 1 1 5D724DEC
-P 4650 3100
-F 0 "R1" H 4720 3146 50  0001 L CNN
-F 1 "4K7" H 4720 3100 50  0000 L CNN
-F 2 "Resistor_THT:R_Axial_DIN0207_L6.3mm_D2.5mm_P10.16mm_Horizontal" V 4580 3100 50  0001 C CNN
-F 3 "~" H 4650 3100 50  0001 C CNN
-	1    4650 3100
-	1    0    0    -1
-$EndComp
-Wire Wire Line
-	4650 2950 4650 2850
-Connection ~ 4650 2850
-Wire Wire Line
-	4650 3250 4650 3400
-Wire Wire Line
-	4650 3400 4500 3400
-Wire Wire Line
-	4500 3400 4500 3100
-$Comp
 L Regulator_Linear:L7805 U4
 U 1 1 5D742D1A
@@
 Connection ~ 5150 1700
 Wire Wire Line
-	5150 1700 3400 1700
+	5150 1700 4850 1700
 Wire Wire Line
 	6050 1900 6050 1700
@@
 Connection ~ 3900 2850
 Wire Wire Line
-	3900 2850 4650 2850
-Wire Wire Line
 	3300 3350 3300 4350
 Wire Wire Line
@@
 Wire Wire Line
 	4000 5000 3650 5000
-Wire Wire Line
-	3650 5200 4500 5200
-Wire Wire Line
-	4500 5200 4500 3400
-Connection ~ 4500 3400
 $Comp
 L Connector_Generic:Conn_01x04 J4
@@
 Wire Wire Line
 	5900 3900 5900 4100
+Wire Wire Line
+	3900 2850 4750 2850
+$Comp
+L Connector_Generic:Conn_01x03 J?
+U 1 1 5D733E64
+P 4550 3050
+F 0 "J?" V 4514 2862 50  0001 R CNN
+F 1 "DS18B20" V 4468 2862 50  0000 R CNN
+F 2 "" H 4550 3050 50  0001 C CNN
+F 3 "~" H 4550 3050 50  0001 C CNN
+	1    4550 3050
+	0    -1   -1   0
+$EndComp
+Wire Wire Line
+	3650 5200 4550 5200
+Wire Wire Line
+	4650 3250 4750 3250
+Wire Wire Line
+	4750 3250 4750 2850
+Connection ~ 4750 2850
+$Comp
+L power:GND #PWR?
+U 1 1 5D73A841
+P 4350 3400
+F 0 "#PWR?" H 4350 3150 50  0001 C CNN
+F 1 "GND" H 4355 3227 50  0000 C CNN
+F 2 "" H 4350 3400 50  0001 C CNN
+F 3 "" H 4350 3400 50  0001 C CNN
+	1    4350 3400
+	1    0    0    -1
+$EndComp
+Wire Wire Line
+	4450 3250 4350 3250
+Wire Wire Line
+	4350 3250 4350 3400
+Wire Wire Line
+	1800 1850 1800 1900
+Wire Wire Line
+	1800 1900 1900 1900
+Connection ~ 1900 1900
+Wire Wire Line
+	4550 3250 4550 5200
+$Comp
+L Connector_Generic:Conn_01x04 J?
+U 1 1 5D75939C
+P 5550 4550
+F 0 "J?" H 5630 4542 50  0001 L CNN
+F 1 "4pin FAN" H 5630 4496 50  0000 L CNN
+F 2 "Connector:FanPinHeader_1x04_P2.54mm_Vertical" H 5550 4550 50  0001 C CNN
+F 3 "~" H 5550 4550 50  0001 C CNN
+	1    5550 4550
+	1    0    0    -1
+$EndComp
+$Comp
+L Connector_Generic:Conn_01x04 J?
+U 1 1 5D75AEB3
+P 5550 5050
+F 0 "J?" H 5630 5042 50  0001 L CNN
+F 1 "4pin FAN" H 5630 4996 50  0000 L CNN
+F 2 "Connector:FanPinHeader_1x04_P2.54mm_Vertical" H 5550 5050 50  0001 C CNN
+F 3 "~" H 5550 5050 50  0001 C CNN
+	1    5550 5050
+	1    0    0    -1
+$EndComp
+$Comp
+L Connector_Generic:Conn_01x04 J?
+U 1 1 5D75B498
+P 5550 5550
+F 0 "J?" H 5630 5542 50  0001 L CNN
+F 1 "4pin FAN" H 5630 5496 50  0000 L CNN
+F 2 "Connector:FanPinHeader_1x04_P2.54mm_Vertical" H 5550 5550 50  0001 C CNN
+F 3 "~" H 5550 5550 50  0001 C CNN
+	1    5550 5550
+	1    0    0    -1
+$EndComp
+$Comp
+L power:GND #PWR?
+U 1 1 5D75BBF3
+P 5200 4350
+F 0 "#PWR?" H 5200 4100 50  0001 C CNN
+F 1 "GND" H 5205 4177 50  0000 C CNN
+F 2 "" H 5200 4350 50  0001 C CNN
+F 3 "" H 5200 4350 50  0001 C CNN
+	1    5200 4350
+	1    0    0    -1
+$EndComp
+$Comp
+L power:GND #PWR?
+U 1 1 5D75C551
+P 5200 4850
+F 0 "#PWR?" H 5200 4600 50  0001 C CNN
+F 1 "GND" H 5205 4677 50  0000 C CNN
+F 2 "" H 5200 4850 50  0001 C CNN
+F 3 "" H 5200 4850 50  0001 C CNN
+	1    5200 4850
+	1    0    0    -1
+$EndComp
+$Comp
+L power:GND #PWR?
+U 1 1 5D75CAEA
+P 5200 5350
+F 0 "#PWR?" H 5200 5100 50  0001 C CNN
+F 1 "GND" H 5205 5177 50  0000 C CNN
+F 2 "" H 5200 5350 50  0001 C CNN
+F 3 "" H 5200 5350 50  0001 C CNN
+	1    5200 5350
+	1    0    0    -1
+$EndComp
+Wire Wire Line
+	5350 4450 5350 4350
+Wire Wire Line
+	5350 4350 5200 4350
+Wire Wire Line
+	5350 4950 5350 4850
+Wire Wire Line
+	5350 4850 5200 4850
+Wire Wire Line
+	5350 5450 5350 5350
+Wire Wire Line
+	5350 5350 5200 5350
+Wire Wire Line
+	5350 5550 4850 5550
+Wire Wire Line
+	4850 5550 4850 5050
+Connection ~ 4850 1700
+Wire Wire Line
+	4850 1700 3400 1700
+Wire Wire Line
+	5350 5050 4850 5050
+Connection ~ 4850 5050
+Wire Wire Line
+	4850 5050 4850 4550
+Wire Wire Line
+	5350 4550 4850 4550
+Connection ~ 4850 4550
+Wire Wire Line
+	4850 4550 4850 1700
+Wire Wire Line
+	3650 5300 4650 5300
+Wire Wire Line
+	4650 5300 4650 4750
+Wire Wire Line
+	4650 4750 5350 4750
+Wire Wire Line
+	3650 5400 4750 5400
+Wire Wire Line
+	4750 5400 4750 5250
+Wire Wire Line
+	4750 5250 5350 5250
+Wire Wire Line
+	3650 5500 4750 5500
+Wire Wire Line
+	4750 5500 4750 5750
+Wire Wire Line
+	4750 5750 5350 5750
 $EndSCHEMATC
