File: PCB/PCB.kicad_pcb (KiCad board)
At the start: 2 copper layers, 1 part

Commit message: PCB update
Parts:
- removed REF**: ESP32-WROOM-32, RF_Module:ESP32-WROOM-32
Changed lines of the file:
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@@
     (tracks 0)
     (zones 0)
-    (modules 1)
+    (modules 0)
     (nets 1)
   )
@@
     (uvia_drill 0.1)
   )
-  (module RF_Module:ESP32-WROOM-32 (layer F.Cu)
-    (at 133.35 101.6)
-    (descr "Single 2.4 GHz Wi-Fi and Bluetooth combo chip https://www.espressif.com/sites/default/files/documentation/esp32-wroom-32_datasheet_en.pdf")
-    (tags "Single 2.4 GHz Wi-Fi and Bluetooth combo  chip")
-    (attr smd)
-    (fp_text reference REF** (at -10.61 8.43 90) (layer F.SilkS)
-      (effects (font (size 1 1) (thickness 0.15)))
-    )
-    (fp_text value ESP32-WROOM-32 (at 0 11.5) (layer F.Fab)
-      (effects (font (size 1 1) (thickness 0.15)))
-    )
-    (fp_line (start -9.12 -9.445) (end -9.5 -9.445) (layer F.SilkS) (width 0.12))
-    (fp_line (start -9.12 -15.865) (end -9.12 -9.445) (layer F.SilkS) (width 0.12))
-    (fp_line (start 9.12 -15.865) (end 9.12 -9.445) (layer F.SilkS) (width 0.12))
-    (fp_line (start -9.12 -15.865) (end 9.12 -15.865) (layer F.SilkS) (width 0.12))
-    (fp_line (start 9.12 9.88) (end 8.12 9.88) (layer F.SilkS) (width 0.12))
-    (fp_line (start 9.12 9.1) (end 9.12 9.88) (layer F.SilkS) (width 0.12))
-    (fp_line (start -9.12 9.88) (end -8.12 9.88) (layer F.SilkS) (width 0.12))
-    (fp_line (start -9.12 9.1) (end -9.12 9.88) (layer F.SilkS) (width 0.12))
-    (fp_line (start 8.4 -20.6) (end 8.2 -20.4) (layer Cmts.User) (width 0.1))
-    (fp_line (start 8.4 -16) (end 8.4 -20.6) (layer Cmts.User) (width 0.1))
-    (fp_line (start 8.4 -20.6) (end 8.6 -20.4) (layer Cmts.User) (width 0.1))
-    (fp_line (start 8.4 -16) (end 8.6 -16.2) (layer Cmts.User) (width 0.1))
-    (fp_line (start 8.4 -16) (end 8.2 -16.2) (layer Cmts.User) (width 0.1))
-    (fp_line (start -9.2 -13.875) (end -9.4 -14.075) (layer Cmts.User) (width 0.1))
-    (fp_line (start -13.8 -13.875) (end -9.2 -13.875) (layer Cmts.User) (width 0.1))
-    (fp_line (start -9.2 -13.875) (end -9.4 -13.675) (layer Cmts.User) (width 0.1))
-    (fp_line (start -13.8 -13.875) (end -13.6 -13.675) (layer Cmts.User) (width 0.1))
-    (fp_line (start -13.8 -13.875) (end -13.6 -14.075) (layer Cmts.User) (width 0.1))
-    (fp_line (start 9.2 -13.875) (end 9.4 -13.675) (layer Cmts.User) (width 0.1))
-    (fp_line (start 9.2 -13.875) (end 9.4 -14.075) (layer Cmts.User) (width 0.1))
-    (fp_line (start 13.8 -13.875) (end 13.6 -13.675) (layer Cmts.User) (width 0.1))
-    (fp_line (start 13.8 -13.875) (end 13.6 -14.075) (layer Cmts.User) (width 0.1))
-    (fp_line (start 9.2 -13.875) (end 13.8 -13.875) (layer Cmts.User) (width 0.1))
-    (fp_line (start 14 -11.585) (end 12 -9.97) (layer Dwgs.User) (width 0.1))
-    (fp_line (start 14 -13.2) (end 10 -9.97) (layer Dwgs.User) (width 0.1))
-    (fp_line (start 14 -14.815) (end 8 -9.97) (layer Dwgs.User) (width 0.1))
-    (fp_line (start 14 -16.43) (end 6 -9.97) (layer Dwgs.User) (width 0.1))
-    (fp_line (start 14 -18.045) (end 4 -9.97) (layer Dwgs.User) (width 0.1))
-    (fp_line (start 14 -19.66) (end 2 -9.97) (layer Dwgs.User) (width 0.1))
-    (fp_line (start 13.475 -20.75) (end 0 -9.97) (layer Dwgs.User) (width 0.1))
-    (fp_line (start 11.475 -20.75) (end -2 -9.97) (layer Dwgs.User) (width 0.1))
-    (fp_line (start 9.475 -20.75) (end -4 -9.97) (layer Dwgs.User) (width 0.1))
-    (fp_line (start 7.475 -20.75) (end -6 -9.97) (layer Dwgs.User) (width 0.1))
-    (fp_line (start -8 -9.97) (end 5.475 -20.75) (layer Dwgs.User) (width 0.1))
-    (fp_line (start 3.475 -20.75) (end -10 -9.97) (layer Dwgs.User) (width 0.1))
-    (fp_line (start 1.475 -20.75) (end -12 -9.97) (layer Dwgs.User) (width 0.1))
-    (fp_line (start -0.525 -20.75) (end -14 -9.97) (layer Dwgs.User) (width 0.1))
-    (fp_line (start -2.525 -20.75) (end -14 -11.585) (layer Dwgs.User) (width 0.1))
-    (fp_line (start -4.525 -20.75) (end -14 -13.2) (layer Dwgs.User) (width 0.1))
-    (fp_line (start -6.525 -20.75) (end -14 -14.815) (layer Dwgs.User) (width 0.1))
-    (fp_line (start -8.525 -20.75) (end -14 -16.43) (layer Dwgs.User) (width 0.1))
-    (fp_line (start -10.525 -20.75) (end -14 -18.045) (layer Dwgs.User) (width 0.1))
-    (fp_line (start -12.525 -20.75) (end -14 -19.66) (layer Dwgs.User) (width 0.1))
-    (fp_line (start 9.75 -9.72) (end 14.25 -9.72) (layer F.CrtYd) (width 0.05))
-    (fp_line (start -14.25 -9.72) (end -9.75 -9.72) (layer F.CrtYd) (width 0.05))
-    (fp_line (start 14.25 -21) (end 14.25 -9.72) (layer F.CrtYd) (width 0.05))
-    (fp_line (start -14.25 -21) (end -14.25 -9.72) (layer F.CrtYd) (width 0.05))
-    (fp_line (start 14 -20.75) (end -14 -20.75) (layer Dwgs.User) (width 0.1))
-    (fp_line (start 14 -9.97) (end 14 -20.75) (layer Dwgs.User) (width 0.1))
-    (fp_line (start 14 -9.97) (end -14 -9.97) (layer Dwgs.User) (width 0.1))
-    (fp_line (start -9 -9.02) (end -8.5 -9.52) (layer F.Fab) (width 0.1))
-    (fp_line (start -8.5 -9.52) (end -9 -10.02) (layer F.Fab) (width 0.1))
-    (fp_line (start -9 -9.02) (end -9 9.76) (layer F.Fab) (width 0.1))
-    (fp_line (start -14.25 -21) (end 14.25 -21) (layer F.CrtYd) (width 0.05))
-    (fp_line (start 9.75 -9.72) (end 9.75 10.5) (layer F.CrtYd) (width 0.05))
-    (fp_line (start -9.75 10.5) (end 9.75 10.5) (layer F.CrtYd) (width 0.05))
-    (fp_line (start -9.75 10.5) (end -9.75 -9.72) (layer F.CrtYd) (width 0.05))
-    (fp_line (start -9 -15.745) (end 9 -15.745) (layer F.Fab) (width 0.1))
-    (fp_line (start -9 -15.745) (end -9 -10.02) (layer F.Fab) (width 0.1))
-    (fp_line (start -9 9.76) (end 9 9.76) (layer F.Fab) (width 0.1))
-    (fp_line (start 9 9.76) (end 9 -15.745) (layer F.Fab) (width 0.1))
-    (fp_line (start -14 -9.97) (end -14 -20.75) (layer Dwgs.User) (width 0.1))
-    (fp_text user "5 mm" (at 7.8 -19.075 90) (layer Cmts.User)
-      (effects (font (size 0.5 0.5) (thickness 0.1)))
-    )
-    (fp_text user "5 mm" (at -11.2 -14.375) (layer Cmts.User)
-      (effects (font (size 0.5 0.5) (thickness 0.1)))
-    )
-    (fp_text user "5 mm" (at 11.8 -14.375) (layer Cmts.User)
-      (effects (font (size 0.5 0.5) (thickness 0.1)))
-    )
-    (fp_text user Antenna (at 0 -13) (layer Cmts.User)
-      (effects (font (size 1 1) (thickness 0.15)))
-    )
-    (fp_text user "KEEP-OUT ZONE" (at 0 -19) (layer Cmts.User)
-      (effects (font (size 1 1) (thickness 0.15)))
-    )
-    (fp_text user %R (at 0 0) (layer F.Fab)
-      (effects (font (size 1 1) (thickness 0.15)))
-    )
-    (pad 38 smd rect (at 8.5 -8.255) (size 2 0.9) (layers F.Cu F.Paste F.Mask))
-    (pad 37 smd rect (at 8.5 -6.985) (size 2 0.9) (layers F.Cu F.Paste F.Mask))
-    (pad 36 smd rect (at 8.5 -5.715) (size 2 0.9) (layers F.Cu F.Paste F.Mask))
-    (pad 35 smd rect (at 8.5 -4.445) (size 2 0.9) (layers F.Cu F.Paste F.Mask))
-    (pad 34 smd rect (at 8.5 -3.175) (size 2 0.9) (layers F.Cu F.Paste F.Mask))
-    (pad 33 smd rect (at 8.5 -1.905) (size 2 0.9) (layers F.Cu F.Paste F.Mask))
-    (pad 32 smd rect (at 8.5 -0.635) (size 2 0.9) (layers F.Cu F.Paste F.Mask))
-    (pad 31 smd rect (at 8.5 0.635) (size 2 0.9) (layers F.Cu F.Paste F.Mask))
-    (pad 30 smd rect (at 8.5 1.905) (size 2 0.9) (layers F.Cu F.Paste F.Mask))
-    (pad 29 smd rect (at 8.5 3.175) (size 2 0.9) (layers F.Cu F.Paste F.Mask))
-    (pad 28 smd rect (at 8.5 4.445) (size 2 0.9) (layers F.Cu F.Paste F.Mask))
-    (pad 27 smd rect (at 8.5 5.715) (size 2 0.9) (layers F.Cu F.Paste F.Mask))
-    (pad 26 smd rect (at 8.5 6.985) (size 2 0.9) (layers F.Cu F.Paste F.Mask))
-    (pad 25 smd rect (at 8.5 8.255) (size 2 0.9) (layers F.Cu F.Paste F.Mask))
-    (pad 24 smd rect (at 5.715 9.255 90) (size 2 0.9) (layers F.Cu F.Paste F.Mask))
-    (pad 23 smd rect (at 4.445 9.255 90) (size 2 0.9) (layers F.Cu F.Paste F.Mask))
-    (pad 22 smd rect (at 3.175 9.255 90) (size 2 0.9) (layers F.Cu F.Paste F.Mask))
-    (pad 21 smd rect (at 1.905 9.255 90) (size 2 0.9) (layers F.Cu F.Paste F.Mask))
-    (pad 20 smd rect (at 0.635 9.255 90) (size 2 0.9) (layers F.Cu F.Paste F.Mask))
-    (pad 19 smd rect (at -0.635 9.255 90) (size 2 0.9) (layers F.Cu F.Paste F.Mask))
-    (pad 18 smd rect (at -1.905 9.255 90) (size 2 0.9) (layers F.Cu F.Paste F.Mask))
-    (pad 17 smd rect (at -3.175 9.255 90) (size 2 0.9) (layers F.Cu F.Paste F.Mask))
-    (pad 16 smd rect (at -4.445 9.255 90) (size 2 0.9) (layers F.Cu F.Paste F.Mask))
-    (pad 15 smd rect (at -5.715 9.255 90) (size 2 0.9) (layers F.Cu F.Paste F.Mask))
-    (pad 14 smd rect (at -8.5 8.255) (size 2 0.9) (layers F.Cu F.Paste F.Mask))
-    (pad 13 smd rect (at -8.5 6.985) (size 2 0.9) (layers F.Cu F.Paste F.Mask))
-    (pad 12 smd rect (at -8.5 5.715) (size 2 0.9) (layers F.Cu F.Paste F.Mask))
-    (pad 11 smd rect (at -8.5 4.445) (size 2 0.9) (layers F.Cu F.Paste F.Mask))
-    (pad 10 smd rect (at -8.5 3.175) (size 2 0.9) (layers F.Cu F.Paste F.Mask))
-    (pad 9 smd rect (at -8.5 1.905) (size 2 0.9) (layers F.Cu F.Paste F.Mask))
-    (pad 8 smd rect (at -8.5 0.635) (size 2 0.9) (layers F.Cu F.Paste F.Mask))
-    (pad 7 smd rect (at -8.5 -0.635) (size 2 0.9) (layers F.Cu F.Paste F.Mask))
-    (pad 6 smd rect (at -8.5 -1.905) (size 2 0.9) (layers F.Cu F.Paste F.Mask))
-    (pad 5 smd rect (at -8.5 -3.175) (size 2 0.9) (layers F.Cu F.Paste F.Mask))
-    (pad 4 smd rect (at -8.5 -4.445) (size 2 0.9) (layers F.Cu F.Paste F.Mask))
-    (pad 3 smd rect (at -8.5 -5.715) (size 2 0.9) (layers F.Cu F.Paste F.Mask))
-    (pad 2 smd rect (at -8.5 -6.985) (size 2 0.9) (layers F.Cu F.Paste F.Mask))
-    (pad 1 smd rect (at -8.5 -8.255) (size 2 0.9) (layers F.Cu F.Paste F.Mask))
-    (pad 39 smd rect (at -1 -0.755) (size 5 5) (layers F.Cu F.Paste F.Mask))
-    (model ${KISYS3DMOD}/RF_Module.3dshapes/ESP32-WROOM-32.wrl
-      (at (xyz 0 0 0))
-      (scale (xyz 1 1 1))
-      (rotate (xyz 0 0 0))
-    )
-  )
 )

Commit message: PCB reated #4
Parts:
- added 0.1uF: , Capacitor_SMD:C_1206_3216Metric, F.Cu at (202.6, 88.3)
- added 0.1uF: , Capacitor_SMD:C_1206_3216Metric, F.Cu at (168.9, 66.0)
- added 0.33uF: , Capacitor_SMD:C_1206_3216Metric, F.Cu at (216.5, 89.5)
- added 12MHz: , Crystal:Crystal_HC49-U_Vertical, F.Cu at (146.1, 76.8)
- added 2.2uF: , Capacitor_THT:CP_Radial_D5.0mm_P2.00mm, F.Cu at (154.9, 58.4)
- added 22pF: , Capacitor_SMD:C_1206_3216Metric, F.Cu at (152.4, 69.2)
- added 22pF: , Capacitor_SMD:C_1206_3216Metric, F.Cu at (148.0, 69.2)
- added 5k6: , Resistor_THT:R_Axial_DIN0207_L6.3mm_D2.5mm_P10.16mm_Horizontal, F.Cu at (158.8, 83.8)
- added 5k6: , Resistor_THT:R_Axial_DIN0207_L6.3mm_D2.5mm_P10.16mm_Horizontal, F.Cu at (216.5, 110.5)
- added 5k6: , Resistor_THT:R_Axial_DIN0207_L6.3mm_D2.5mm_P10.16mm_Horizontal, F.Cu at (198.8, 110.5)
- added 5k6: , Resistor_THT:R_Axial_DIN0207_L6.3mm_D2.5mm_P10.16mm_Horizontal, F.Cu at (150.5, 110.5)
- added 5k6: , Resistor_THT:R_Axial_DIN0207_L6.3mm_D2.5mm_P10.16mm_Horizontal, F.Cu at (134.6, 110.5)
- added 5k6: , Resistor_THT:R_Axial_DIN0207_L6.3mm_D2.5mm_P10.16mm_Horizontal, F.Cu at (183.5, 110.5)
- added 5k6: , Resistor_THT:R_Axial_DIN0207_L6.3mm_D2.5mm_P10.16mm_Horizontal, F.Cu at (165.7, 110.5)
- added CH340G: , Package_SO:SOP-16_4.4x10.4mm_P1.27mm, F.Cu at (160.7, 74.9)
- added DS18B20: , Connector_PinHeader_2.54mm:PinHeader_1x03_P2.54mm_Horizontal, F.Cu at (221.6, 55.9)
- added ESP32-WROOM-32: , RF_Module:ESP32-WROOM-32, F.Cu at (182.2, 64.1)
- added FAN 1: , Connector:FanPinHeader_1x04_P2.54mm_Vertical, F.Cu at (214.6, 56.5)
- added FAN 2: , Connector:FanPinHeader_1x04_P2.54mm_Vertical, F.Cu at (214.6, 66.0)
- added FAN 3: , Connector:FanPinHeader_1x04_P2.54mm_Vertical, F.Cu at (214.6, 75.6)
- added IRF530N: , Package_TO_SOT_THT:TO-220-3_Vertical, F.Cu at (152.4, 85.1)
- added IRF530N: , Package_TO_SOT_THT:TO-220-3_Vertical, F.Cu at (221.0, 110.5)
- added IRF530N: , Package_TO_SOT_THT:TO-220-3_Vertical, F.Cu at (203.2, 110.5)
- added IRF530N: , Package_TO_SOT_THT:TO-220-3_Vertical, F.Cu at (154.9, 110.5)
- added IRF530N: , Package_TO_SOT_THT:TO-220-3_Vertical, F.Cu at (139.1, 110.5)
- added IRF530N: , Package_TO_SOT_THT:TO-220-3_Vertical, F.Cu at (188.0, 110.5)
- added IRF530N: , Package_TO_SOT_THT:TO-220-3_Vertical, F.Cu at (170.2, 110.5)
- added IRFD110: , Package_DIP:Vishay_HVM-DIP-3_W7.62mm, F.Cu at (163.2, 91.4)
- added IRFD110: , Package_DIP:Vishay_HVM-DIP-3_W7.62mm, F.Cu at (228.6, 102.9)
- added IRFD110: , Package_DIP:Vishay_HVM-DIP-3_W7.62mm, F.Cu at (210.8, 102.9)
- added IRFD110: , Package_DIP:Vishay_HVM-DIP-3_W7.62mm, F.Cu at (162.6, 102.9)
- added IRFD110: , Package_DIP:Vishay_HVM-DIP-3_W7.62mm, F.Cu at (146.7, 102.9)
- added IRFD110: , Package_DIP:Vishay_HVM-DIP-3_W7.62mm, F.Cu at (195.6, 102.9)
- added IRFD110: , Package_DIP:Vishay_HVM-DIP-3_W7.62mm, F.Cu at (177.8, 102.9)
- added IRFD110: , Package_DIP:Vishay_HVM-DIP-3_W7.62mm, F.Cu at (185.4, 92.1)
- added L7805: , Package_TO_SOT_SMD:TO-252-2, F.Cu at (210.2, 89.5)
- added LF33CDT: , Package_TO_SOT_SMD:TO-252-2, F.Cu at (165.1, 59.7)
- added NEXTION 2.8": , Connector_PinHeader_2.54mm:PinHeader_1x04_P2.54mm_Horizontal, F.Cu at (221.6, 66.7)
- added Peltiers 12V: , Connector_Phoenix_GMSTB:PhoenixContact_GMSTBVA_2,5_4-G-7,62_1x04_P7.62mm_Vertical, F.Cu at (170.2, 120.7)
- added Peltiers 3.3V: , Connector_Phoenix_GMSTB:PhoenixContact_GMSTBVA_2,5_4-G-7,62_1x04_P7.62mm_Vertical, F.Cu at (137.2, 120.7)
- added REF**: KiCad-Logo2_6mm_SilkScreen, Symbol:KiCad-Logo2_6mm_SilkScreen, F.Cu at (197.5, 69.8)
- added REF**: KiCad-Logo2_20mm_SilkScreen, Symbol:KiCad-Logo2_20mm_SilkScreen, B.Cu at (179.7, 73.7)
- added REF**: WEEE-Logo_8.4x12mm_SilkScreen, Symbol:WEEE-Logo_8.4x12mm_SilkScreen, F.Cu at (194.3, 87.6)
- added REF**: RoHS-Logo_6mm_SilkScreen, Symbol:RoHS-Logo_6mm_SilkScreen, B.Cu at (208.3, 91.4)
- added REF**: MountingHole_3.2mm_M3_Pad_Via, MountingHole:MountingHole_3.2mm_M3_Pad_Via, F.Cu at (138.4, 76.2)
- added REF**: MountingHole_3.2mm_M3_Pad_Via, MountingHole:MountingHole_3.2mm_M3_Pad_Via, F.Cu at (225.4, 92.1)
- added REF**: MountingHole_3.2mm_M3_Pad_Via, MountingHole:MountingHole_3.2mm_M3_Pad_Via, F.Cu at (199.4, 55.9)
- added USB_B: , Connector_USB:USB_B_OST_USB-B1HSxx_Horizontal, F.Cu at (142.9, 64.1)
- added Vapor maker: , Connector_Phoenix_GMSTB:PhoenixContact_GMSTBVA_2,5_4-G-7,62_1x04_P7.62mm_Vertical, F.Cu at (203.2, 120.7)
- added chamber LED: , TerminalBlock_WAGO:TerminalBlock_WAGO_804-102_1x02_P5.00mm_45Degree, F.Cu at (141.0, 85.1)
- added power 12V: , Connector_PinHeader_2.54mm:PinHeader_1x03_P2.54mm_Horizontal, F.Cu at (221.6, 80.6)
Routing:
- net (no net): track 0.00 -> 166.2 mm
- net Net-(C4-Pad1): track 0.00 -> 130.8 mm, vias 0 -> 3
- net GND: track 0.00 -> 117.2 mm, vias 0 -> 21
- net Net-(C3-Pad1): track 0.00 -> 116.4 mm, vias 0 -> 3
- net Net-(Q10-Pad1): track 0.00 -> 115.2 mm
- net Net-(Q13-Pad2): track 0.00 -> 66.4 mm
- net Net-(Q10-Pad2): track 0.00 -> 64.7 mm
- net Net-(J3-Pad2): track 0.00 -> 61.6 mm, vias 0 -> 2
- net Net-(J4-Pad3): track 0.00 -> 57.5 mm, vias 0 -> 2
- net Net-(Q12-Pad2): track 0.00 -> 56.3 mm
- net Net-(J4-Pad2): track 0.00 -> 55.8 mm, vias 0 -> 2
- net Net-(Q11-Pad2): track 0.00 -> 53.4 mm, vias 0 -> 2
- net Net-(Q9-Pad2): track 0.00 -> 52.9 mm, vias 0 -> 2
- net Net-(Q8-Pad2): track 0.00 -> 44.9 mm, vias 0 -> 2
- net Net-(Q7-Pad2): track 0.00 -> 32.7 mm, vias 0 -> 2
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- added copper zone on B.Cu, net GND
- added copper zone on F.Cu, net GND
Other:
- board outline added: 99.1 x 74.3 mm
- board text added: "12V"
- board text added: "3V3"
- board text added: "5V"
- board text added: "D1"
- board text added: "GND"
- board text added: "RXD"
- board text added: "TXD"

Commit message: gerbers created
Routing:
- net GND: vias 21 -> 23
Changed lines of the file:
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@@
     (thickness 1.6)
     (drawings 30)
-    (tracks 526)
+    (tracks 528)
     (zones 0)
     (modules 51)
@@
   (page A4)
   (layers
-    (0 F.Cu signal hide)
-    (31 B.Cu signal hide)
+    (0 F.Cu signal)
+    (31 B.Cu signal)
     (32 B.Adhes user)
     (33 F.Adhes user)
     (34 B.Paste user)
     (35 F.Paste user)
-    (36 B.SilkS user)
-    (37 F.SilkS user)
+    (36 B.SilkS user hide)
+    (37 F.SilkS user hide)
     (38 B.Mask user)
     (39 F.Mask user)
@@
   )
   (setup
-    (last_trace_width 2)
+    (last_trace_width 0.25)
     (user_trace_width 0.5)
     (user_trace_width 0.75)
@@
     (visible_elements FFFFF77F)
     (pcbplotparams
-      (layerselection 0x010fc_ffffffff)
+      (layerselection 0x010f0_ffffffff)
       (usegerberextensions false)
       (usegerberattributes false)
@@
       (outputformat 1)
       (mirror false)
-      (drillshape 1)
+      (drillshape 0)
       (scaleselection 1)
-      (outputdirectory ""))
+      (outputdirectory "gerber/"))
   )
   (net 0 "")
@@
   (segment (start 143.47 92.59) (end 140.97 90.09) (width 5) (layer F.Cu) (net 1))
   (segment (start 145.97 92.59) (end 143.47 92.59) (width 5) (layer F.Cu) (net 1))
+  (via (at 170.18 78.74) (size 0.8) (drill 0.4) (layers F.Cu B.Cu) (net 1))
+  (via (at 165.1 67.056) (size 0.8) (drill 0.4) (layers F.Cu B.Cu) (net 1))
   (segment (start 157.48 71.785) (end 157.485 71.78) (width 0.5) (layer F.Cu) (net 2))
   (segment (start 147.955 74.93) (end 147.955 70.615) (width 0.5) (layer F.Cu) (net 2))
