File: PCB/PCB.kicad_pcb (KiCad board)
At the start: 2 copper layers, 121.4 x 90.9 mm, 88 parts, among them J1 GND, J10 VM1, J11 GND, J12 VM2, J13 GND, J14 P3B, J15 GND, J16 P3A, J17 NEXTION, J18 Power, J19 OneWire, J2 pump, J20 I2C, J3 GND, J4 LED, J5 GND, J6 P12B, J7 GND, J8 P12A, J9 GND, Q1 S8050, Q10 IRLR2905, Q2 S8050, Q3 IRLR2905, Q4 IRLR2905, Q5 IRLR2905, Q6 IRLR2905, Q7 IRLR2905, Q8 IRLR2905, Q9 IRLR2905, X1 12MHz

Commit message: gerber #4
Routing:
- net GND: vias 40 -> 57
- added copper zone on B.Cu, net GND
- added copper zone on F.Cu, net GND
Changed lines of the file:
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@@
   (general
     (thickness 1.6)
-    (drawings 32)
-    (tracks 833)
+    (drawings 30)
+    (tracks 850)
     (zones 0)
     (modules 88)
@@
   (page A4)
   (layers
-    (0 F.Cu signal)
+    (0 F.Cu signal hide)
     (31 B.Cu signal)
     (32 B.Adhes user)
@@
     (36 B.SilkS user)
     (37 F.SilkS user)
-    (38 B.Mask user hide)
-    (39 F.Mask user)
+    (38 B.Mask user)
+    (39 F.Mask user hide)
     (40 Dwgs.User user hide)
     (41 Cmts.User user hide)
@@
       (outputformat 1)
       (mirror false)
-      (drillshape 1)
+      (drillshape 0)
       (scaleselection 1)
-      (outputdirectory ""))
+      (outputdirectory "gerber/"))
   )
   (net 0 "")
@@
     (effects (font (size 1.3 1.3) (thickness 0.3)))
   )
-  (gr_poly (pts (xy 145.034 64.77) (xy 144.526 64.008) (xy 144.526 60.96) (xy 145.034 60.198)) (layer B.Mask) (width 0.1))
-  (gr_poly (pts (xy 129.794 68.58) (xy 129.286 67.818) (xy 129.286 64.77) (xy 129.794 64.008)) (layer B.Mask) (width 0.1))
   (gr_line (start 86.614 45.974) (end 208.026 45.974) (layer Edge.Cuts) (width 0.05))
   (dimension 90.932 (width 0.15) (layer Cmts.User)
@@
   (segment (start 111.76 111.76) (end 111.76 108.975001) (width 4.5) (layer F.Cu) (net 1))
   (segment (start 98.705 114.655) (end 98.705 108.975001) (width 4.5) (layer F.Cu) (net 1))
+  (via (at 170.18 90.17) (size 0.8) (drill 0.4) (layers F.Cu B.Cu) (net 1))
+  (via (at 173.99 90.17) (size 0.8) (drill 0.4) (layers F.Cu B.Cu) (net 1))
+  (via (at 165.1 96.52) (size 0.8) (drill 0.4) (layers F.Cu B.Cu) (net 1))
+  (via (at 173.99 96.52) (size 0.8) (drill 0.4) (layers F.Cu B.Cu) (net 1))
+  (via (at 182.88 96.52) (size 0.8) (drill 0.4) (layers F.Cu B.Cu) (net 1))
+  (via (at 193.04 92.71) (size 0.8) (drill 0.4) (layers F.Cu B.Cu) (net 1))
+  (via (at 119.38 85.09) (size 0.8) (drill 0.4) (layers F.Cu B.Cu) (net 1))
+  (via (at 128.27 85.09) (size 0.8) (drill 0.4) (layers F.Cu B.Cu) (net 1))
+  (via (at 162.56 87.63) (size 0.8) (drill 0.4) (layers F.Cu B.Cu) (net 1))
+  (via (at 152.4 87.63) (size 0.8) (drill 0.4) (layers F.Cu B.Cu) (net 1))
+  (via (at 124.46 73.66) (size 0.8) (drill 0.4) (layers F.Cu B.Cu) (net 1))
+  (via (at 119.38 69.85) (size 0.8) (drill 0.4) (layers F.Cu B.Cu) (net 1))
+  (via (at 167.64 67.31) (size 0.8) (drill 0.4) (layers F.Cu B.Cu) (net 1))
+  (via (at 165.1 67.31) (size 0.8) (drill 0.4) (layers F.Cu B.Cu) (net 1))
+  (via (at 166.37 66.04) (size 0.8) (drill 0.4) (layers F.Cu B.Cu) (net 1))
+  (via (at 102.87 59.69) (size 0.8) (drill 0.4) (layers F.Cu B.Cu) (net 1))
+  (via (at 101.6 55.88) (size 0.8) (drill 0.4) (layers F.Cu B.Cu) (net 1))
   (segment (start 200.225 81.28) (end 198.755 82.75) (width 0.75) (layer B.Cu) (net 2))
   (segment (start 204.47 81.28) (end 200.225 81.28) (width 0.75) (layer B.Cu) (net 2))
@@
   (segment (start 185.928 93.98) (end 189.23 90.678) (width 0.254) (layer B.Cu) (net 65))
   (segment (start 158.75 94.488) (end 159.258 93.98) (width 0.254) (layer B.Cu) (net 65))
+  (zone (net 1) (net_name GND) (layer F.Cu) (hatch edge 0.508)
+    (connect_pads (clearance 0.508))
+    (min_thickness 0.254)
+    (fill yes (arc_segments 32) (thermal_gap 0.508) (thermal_bridge_width 0.508))
+    (polygon
+      (pts
+        (xy 208.026 136.906) (xy 86.614 136.906) (xy 86.614 45.974) (xy 208.026 45.974)
+      )
+    )
+  )
+  (zone (net 1) (net_name GND) (layer B.Cu) (hatch edge 0.508)
+    (connect_pads (clearance 0.508))
+    (min_thickness 0.254)
+    (fill yes (arc_segments 32) (thermal_gap 0.508) (thermal_bridge_width 0.508))
+    (polygon
+      (pts
+        (xy 208.026 136.906) (xy 86.614 136.906) (xy 86.614 45.974) (xy 208.026 45.974)
+      )
+    )
+  )
 )

Commit message: gerber regenerate
Routing:
- net GND: vias 57 -> 54
Changed lines of the file:
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@@
     (thickness 1.6)
     (drawings 30)
-    (tracks 850)
+    (tracks 847)
     (zones 0)
     (modules 88)
@@
   (layers
     (0 F.Cu signal hide)
-    (31 B.Cu signal)
+    (31 B.Cu signal hide)
     (32 B.Adhes user)
     (33 F.Adhes user)
-    (34 B.Paste user hide)
+    (34 B.Paste user)
     (35 F.Paste user)
     (36 B.SilkS user)
     (37 F.SilkS user)
     (38 B.Mask user)
-    (39 F.Mask user hide)
-    (40 Dwgs.User user hide)
+    (39 F.Mask user)
+    (40 Dwgs.User user)
     (41 Cmts.User user hide)
     (42 Eco1.User user)
@@
     (44 Edge.Cuts user)
     (45 Margin user)
-    (46 B.CrtYd user hide)
+    (46 B.CrtYd user)
     (47 F.CrtYd user)
     (48 B.Fab user hide)
-    (49 F.Fab user)
+    (49 F.Fab user hide)
   )
   (setup
-    (last_trace_width 0.5)
+    (last_trace_width 0.25)
     (user_trace_width 0.2)
     (user_trace_width 0.254)
@@
       (usegerberadvancedattributes false)
       (creategerberjobfile false)
-      (excludeedgelayer true)
-      (linewidth 0.100000)
+      (excludeedgelayer false)
+      (linewidth 0.150000)
       (plotframeref false)
       (viasonmask false)
       (mode 1)
-      (useauxorigin false)
+      (useauxorigin true)
       (hpglpennumber 1)
       (hpglpenspeed 20)
@@
     (tags "resistor handsolder")
     (attr smd)
-    (fp_text reference R15 (at 0 1.82 -90 unlocked) (layer B.SilkS)
+    (fp_text reference R15 (at 0 1.82 90 unlocked) (layer B.SilkS)
       (effects (font (size 1 1) (thickness 0.15)) (justify mirror))
     )
@@
   (via (at 124.46 73.66) (size 0.8) (drill 0.4) (layers F.Cu B.Cu) (net 1))
   (via (at 119.38 69.85) (size 0.8) (drill 0.4) (layers F.Cu B.Cu) (net 1))
-  (via (at 167.64 67.31) (size 0.8) (drill 0.4) (layers F.Cu B.Cu) (net 1))
-  (via (at 165.1 67.31) (size 0.8) (drill 0.4) (layers F.Cu B.Cu) (net 1))
-  (via (at 166.37 66.04) (size 0.8) (drill 0.4) (layers F.Cu B.Cu) (net 1))
   (via (at 102.87 59.69) (size 0.8) (drill 0.4) (layers F.Cu B.Cu) (net 1))
   (via (at 101.6 55.88) (size 0.8) (drill 0.4) (layers F.Cu B.Cu) (net 1))
