File: PCB/E32CB_R2/PCB.sch (KiCad schematic (older format))
At the start: 82 parts, among them J1 GND, J10 VM1, J11 GND, J12 VM2, J13 GND, J14 P3B, J15 GND, J16 P3A, J17 NEXTION, J18 Power, J19 OneWire, J2 pump, J20 I2C, J21 USB_B, J3 GND, J4 LED, J5 GND, J6 P12B, J7 GND, J8 P12A, J9 GND, Q1 S8050, Q10 IRLR2905, Q2 S8050, Q3 IRLR2905, Q4 IRLR2905, Q5 IRLR2905, Q6 IRLR2905, Q7 IRLR2905, Q8 IRLR2905, Q9 IRLR2905, U1 ESP32-WROOM-32, X1 12MHz

Commit message: pcb update
Parts:
- removed C9: 2.2uF, Capacitor_SMD:CP_Elec_4x5.4, symbol Device:CP
- added C9: 2.2uF, Capacitor_SMD:C_0805_2012Metric_Pad1.15x1.40mm_HandSolder, symbol Device:C
- C1, C2, C3, C6, C8: footprint Capacitors_SMD:C_1206_HandSoldering -> Capacitors_SMD:C_0805_HandSoldering
- C4, C5, C7: footprint Capacitor_SMD:C_1206_3216Metric_Pad1.42x1.75mm_HandSolder -> Capacitor_SMD:C_0805_2012Metric_Pad1.15x1.40mm_HandSolder
- R1, R10, R11, R12, R13, R14, R15, R16, R17, R18, R19, R2, R20, R21, R3, R4, R5, R6, R7, R8, R9: footprint Resistor_SMD:R_1206_3216Metric_Pad1.42x1.75mm_HandSolder -> Resistor_SMD:R_0805_2012Metric_Pad1.15x1.40mm_HandSolder
Changed lines of the file:
@@
 F 0 "C2" V 1300 2450 50  0000 L CNN
 F 1 "22p" V 1350 2250 50  0000 L CNN
-F 2 "Capacitors_SMD:C_1206_HandSoldering" H 1238 2250 50  0001 C CNN
+F 2 "Capacitors_SMD:C_0805_HandSoldering" H 1238 2250 50  0001 C CNN
 F 3 "~" H 1200 2400 50  0001 C CNN
 	1    1200 2400
@@
 F 0 "C1" V 1100 2150 50  0000 L CNN
 F 1 "22p" V 1050 1950 50  0000 L CNN
-F 2 "Capacitors_SMD:C_1206_HandSoldering" H 1238 1950 50  0001 C CNN
+F 2 "Capacitors_SMD:C_0805_HandSoldering" H 1238 1950 50  0001 C CNN
 F 3 "~" H 1200 2100 50  0001 C CNN
 	1    1200 2100
@@
 F 0 "C7" H 7700 3200 50  0000 L CNN
 F 1 "100nF" H 7600 3000 50  0000 L CNN
-F 2 "Capacitor_SMD:C_1206_3216Metric_Pad1.42x1.75mm_HandSolder" H 7888 2950 50  0001 C CNN
+F 2 "Capacitor_SMD:C_0805_2012Metric_Pad1.15x1.40mm_HandSolder" H 7888 2950 50  0001 C CNN
 F 3 "~" H 7850 3100 50  0001 C CNN
 	1    7850 3100
-	1    0    0    -1
-$EndComp
-$Comp
-L Device:CP C9
-U 1 1 5DF1B2ED
-P 8850 3100
-F 0 "C9" H 8900 3200 50  0000 L CNN
-F 1 "2.2uF" H 8900 3000 50  0000 L CNN
-F 2 "Capacitor_SMD:CP_Elec_4x5.4" H 8888 2950 50  0001 C CNN
-F 3 "~" H 8850 3100 50  0001 C CNN
-	1    8850 3100
 	1    0    0    -1
 $EndComp
@@
 F 0 "C6" H 7765 1596 50  0000 L CNN
 F 1 "330nF" H 7765 1505 50  0000 L CNN
-F 2 "Capacitors_SMD:C_1206_HandSoldering" H 7688 1400 50  0001 C CNN
+F 2 "Capacitors_SMD:C_0805_HandSoldering" H 7688 1400 50  0001 C CNN
 F 3 "~" H 7650 1550 50  0001 C CNN
 	1    7650 1550
@@
 F 0 "C8" H 8765 1596 50  0000 L CNN
 F 1 "100nF" H 8765 1505 50  0000 L CNN
-F 2 "Capacitors_SMD:C_1206_HandSoldering" H 8688 1400 50  0001 C CNN
+F 2 "Capacitors_SMD:C_0805_HandSoldering" H 8688 1400 50  0001 C CNN
 F 3 "~" H 8650 1550 50  0001 C CNN
 	1    8650 1550
@@
 F 0 "C3" H 2000 1050 50  0000 R CNN
 F 1 "10nF" H 2000 1200 50  0000 R CNN
-F 2 "Capacitors_SMD:C_1206_HandSoldering" H 2050 1150 50  0001 C CNN
+F 2 "Capacitors_SMD:C_0805_HandSoldering" H 2050 1150 50  0001 C CNN
 F 3 "~" H 2050 1150 50  0001 C CNN
 	1    2050 1150
@@
 F 0 "R3" V 1550 5450 50  0000 L CNN
 F 1 "1k2" V 1350 5450 50  0000 L CNN
-F 2 "Resistor_SMD:R_1206_3216Metric_Pad1.42x1.75mm_HandSolder" H 1450 5550 50  0001 C CNN
+F 2 "Resistor_SMD:R_0805_2012Metric_Pad1.15x1.40mm_HandSolder" H 1450 5550 50  0001 C CNN
 F 3 "~" H 1450 5550 50  0001 C CNN
 	1    1450 5550
@@
 F 0 "R2" V 1150 5500 50  0000 C CNN
 F 1 "1k2" V 1350 5500 50  0000 C CNN
-F 2 "Resistor_SMD:R_1206_3216Metric_Pad1.42x1.75mm_HandSolder" H 1250 5550 50  0001 C CNN
+F 2 "Resistor_SMD:R_0805_2012Metric_Pad1.15x1.40mm_HandSolder" H 1250 5550 50  0001 C CNN
 F 3 "~" H 1250 5550 50  0001 C CNN
 	1    1250 5550
@@
 F 0 "R1" V 900 7200 50  0000 L CNN
 F 1 "4k7" V 800 7200 50  0000 L CNN
-F 2 "Resistor_SMD:R_1206_3216Metric_Pad1.42x1.75mm_HandSolder" H 900 7250 50  0001 C CNN
+F 2 "Resistor_SMD:R_0805_2012Metric_Pad1.15x1.40mm_HandSolder" H 900 7250 50  0001 C CNN
 F 3 "~" H 900 7250 50  0001 C CNN
 	1    900  7250
@@
 F 0 "R4" V 2754 1500 50  0000 C CNN
 F 1 "470R" V 2845 1500 50  0000 C CNN
-F 2 "Resistor_SMD:R_1206_3216Metric_Pad1.42x1.75mm_HandSolder" H 2950 1500 50  0001 C CNN
+F 2 "Resistor_SMD:R_0805_2012Metric_Pad1.15x1.40mm_HandSolder" H 2950 1500 50  0001 C CNN
 F 3 "~" H 2950 1500 50  0001 C CNN
 	1    2950 1500
@@
 F 0 "R5" V 3150 1600 50  0000 C CNN
 F 1 "470R" V 3050 1600 50  0000 C CNN
-F 2 "Resistor_SMD:R_1206_3216Metric_Pad1.42x1.75mm_HandSolder" H 2950 1600 50  0001 C CNN
+F 2 "Resistor_SMD:R_0805_2012Metric_Pad1.15x1.40mm_HandSolder" H 2950 1600 50  0001 C CNN
 F 3 "~" H 2950 1600 50  0001 C CNN
 	1    2950 1600
@@
 F 0 "R6" V 2954 3800 50  0000 C CNN
 F 1 "1k" V 3045 3800 50  0000 C CNN
-F 2 "Resistor_SMD:R_1206_3216Metric_Pad1.42x1.75mm_HandSolder" H 3150 3800 50  0001 C CNN
+F 2 "Resistor_SMD:R_0805_2012Metric_Pad1.15x1.40mm_HandSolder" H 3150 3800 50  0001 C CNN
 F 3 "~" H 3150 3800 50  0001 C CNN
 	1    3150 3800
@@
 F 0 "R7" V 2954 4150 50  0000 C CNN
 F 1 "1k" V 3045 4150 50  0000 C CNN
-F 2 "Resistor_SMD:R_1206_3216Metric_Pad1.42x1.75mm_HandSolder" H 3150 4150 50  0001 C CNN
+F 2 "Resistor_SMD:R_0805_2012Metric_Pad1.15x1.40mm_HandSolder" H 3150 4150 50  0001 C CNN
 F 3 "~" H 3150 4150 50  0001 C CNN
 	1    3150 4150
@@
 F 0 "R10" V 3004 2150 50  0000 C CNN
 F 1 "12k" V 3095 2150 50  0000 C CNN
-F 2 "Resistor_SMD:R_1206_3216Metric_Pad1.42x1.75mm_HandSolder" H 3200 2150 50  0001 C CNN
+F 2 "Resistor_SMD:R_0805_2012Metric_Pad1.15x1.40mm_HandSolder" H 3200 2150 50  0001 C CNN
 F 3 "~" H 3200 2150 50  0001 C CNN
 	1    3200 2150
@@
 F 0 "R11" V 3400 2350 50  0000 C CNN
 F 1 "12k" V 3300 2350 50  0000 C CNN
-F 2 "Resistor_SMD:R_1206_3216Metric_Pad1.42x1.75mm_HandSolder" H 3200 2350 50  0001 C CNN
+F 2 "Resistor_SMD:R_0805_2012Metric_Pad1.15x1.40mm_HandSolder" H 3200 2350 50  0001 C CNN
 F 3 "~" H 3200 2350 50  0001 C CNN
 	1    3200 2350
@@
 F 0 "R12" H 3509 1446 50  0000 L CNN
 F 1 "10k" H 3509 1355 50  0000 L CNN
-F 2 "Resistor_SMD:R_1206_3216Metric_Pad1.42x1.75mm_HandSolder" H 3450 1400 50  0001 C CNN
+F 2 "Resistor_SMD:R_0805_2012Metric_Pad1.15x1.40mm_HandSolder" H 3450 1400 50  0001 C CNN
 F 3 "~" H 3450 1400 50  0001 C CNN
 	1    3450 1400
@@
 F 0 "R13" H 3759 1446 50  0000 L CNN
 F 1 "10k" H 3759 1355 50  0000 L CNN
-F 2 "Resistor_SMD:R_1206_3216Metric_Pad1.42x1.75mm_HandSolder" H 3700 1400 50  0001 C CNN
+F 2 "Resistor_SMD:R_0805_2012Metric_Pad1.15x1.40mm_HandSolder" H 3700 1400 50  0001 C CNN
 F 3 "~" H 3700 1400 50  0001 C CNN
 	1    3700 1400
@@
 F 0 "C4" H 5792 2696 50  0000 L CNN
 F 1 "100nF" H 5792 2605 50  0000 L CNN
-F 2 "Capacitor_SMD:C_1206_3216Metric_Pad1.42x1.75mm_HandSolder" H 5700 2650 50  0001 C CNN
+F 2 "Capacitor_SMD:C_0805_2012Metric_Pad1.15x1.40mm_HandSolder" H 5700 2650 50  0001 C CNN
 F 3 "~" H 5700 2650 50  0001 C CNN
 	1    5700 2650
@@
 F 0 "C5" H 6192 2696 50  0000 L CNN
 F 1 "10uF" H 6192 2605 50  0000 L CNN
-F 2 "Capacitor_SMD:C_1206_3216Metric_Pad1.42x1.75mm_HandSolder" H 6100 2650 50  0001 C CNN
+F 2 "Capacitor_SMD:C_0805_2012Metric_Pad1.15x1.40mm_HandSolder" H 6100 2650 50  0001 C CNN
 F 3 "~" H 6100 2650 50  0001 C CNN
 	1    6100 2650
@@
 F 0 "R19" H 9959 3346 50  0000 L CNN
 F 1 "470R" H 9959 3255 50  0000 L CNN
-F 2 "Resistor_SMD:R_1206_3216Metric_Pad1.42x1.75mm_HandSolder" H 9900 3300 50  0001 C CNN
+F 2 "Resistor_SMD:R_0805_2012Metric_Pad1.15x1.40mm_HandSolder" H 9900 3300 50  0001 C CNN
 F 3 "~" H 9900 3300 50  0001 C CNN
 	1    9900 3300
@@
 F 0 "R18" H 9959 2296 50  0000 L CNN
 F 1 "470R" H 9959 2205 50  0000 L CNN
-F 2 "Resistor_SMD:R_1206_3216Metric_Pad1.42x1.75mm_HandSolder" H 9900 2250 50  0001 C CNN
+F 2 "Resistor_SMD:R_0805_2012Metric_Pad1.15x1.40mm_HandSolder" H 9900 2250 50  0001 C CNN
 F 3 "~" H 9900 2250 50  0001 C CNN
 	1    9900 2250
@@
 F 0 "R17" H 8659 5796 50  0000 L CNN
 F 1 "470R" H 8659 5705 50  0000 L CNN
-F 2 "Resistor_SMD:R_1206_3216Metric_Pad1.42x1.75mm_HandSolder" H 8600 5750 50  0001 C CNN
+F 2 "Resistor_SMD:R_0805_2012Metric_Pad1.15x1.40mm_HandSolder" H 8600 5750 50  0001 C CNN
 F 3 "~" H 8600 5750 50  0001 C CNN
 	1    8600 5750
@@
 F 0 "R16" H 8659 4746 50  0000 L CNN
 F 1 "470R" H 8659 4655 50  0000 L CNN
-F 2 "Resistor_SMD:R_1206_3216Metric_Pad1.42x1.75mm_HandSolder" H 8600 4700 50  0001 C CNN
+F 2 "Resistor_SMD:R_0805_2012Metric_Pad1.15x1.40mm_HandSolder" H 8600 4700 50  0001 C CNN
 F 3 "~" H 8600 4700 50  0001 C CNN
 	1    8600 4700
@@
 F 0 "R21" H 9959 5796 50  0000 L CNN
 F 1 "470R" H 9959 5705 50  0000 L CNN
-F 2 "Resistor_SMD:R_1206_3216Metric_Pad1.42x1.75mm_HandSolder" H 9900 5750 50  0001 C CNN
+F 2 "Resistor_SMD:R_0805_2012Metric_Pad1.15x1.40mm_HandSolder" H 9900 5750 50  0001 C CNN
 F 3 "~" H 9900 5750 50  0001 C CNN
 	1    9900 5750
@@
 F 0 "R20" H 9959 4746 50  0000 L CNN
 F 1 "470R" H 9959 4655 50  0000 L CNN
-F 2 "Resistor_SMD:R_1206_3216Metric_Pad1.42x1.75mm_HandSolder" H 9900 4700 50  0001 C CNN
+F 2 "Resistor_SMD:R_0805_2012Metric_Pad1.15x1.40mm_HandSolder" H 9900 4700 50  0001 C CNN
 F 3 "~" H 9900 4700 50  0001 C CNN
 	1    9900 4700
@@
 F 0 "R15" H 7359 5796 50  0000 L CNN
 F 1 "470R" H 7359 5705 50  0000 L CNN
-F 2 "Resistor_SMD:R_1206_3216Metric_Pad1.42x1.75mm_HandSolder" H 7300 5750 50  0001 C CNN
+F 2 "Resistor_SMD:R_0805_2012Metric_Pad1.15x1.40mm_HandSolder" H 7300 5750 50  0001 C CNN
 F 3 "~" H 7300 5750 50  0001 C CNN
 	1    7300 5750
@@
 F 0 "R14" H 7359 4746 50  0000 L CNN
 F 1 "470R" H 7359 4655 50  0000 L CNN
-F 2 "Resistor_SMD:R_1206_3216Metric_Pad1.42x1.75mm_HandSolder" H 7300 4700 50  0001 C CNN
+F 2 "Resistor_SMD:R_0805_2012Metric_Pad1.15x1.40mm_HandSolder" H 7300 4700 50  0001 C CNN
 F 3 "~" H 7300 4700 50  0001 C CNN
 	1    7300 4700
@@
 F 0 "R8" V 2954 4550 50  0000 C CNN
 F 1 "1k" V 3045 4550 50  0000 C CNN
-F 2 "Resistor_SMD:R_1206_3216Metric_Pad1.42x1.75mm_HandSolder" H 3150 4550 50  0001 C CNN
+F 2 "Resistor_SMD:R_0805_2012Metric_Pad1.15x1.40mm_HandSolder" H 3150 4550 50  0001 C CNN
 F 3 "~" H 3150 4550 50  0001 C CNN
 	1    3150 4550
@@
 F 0 "R9" V 2954 4950 50  0000 C CNN
 F 1 "1k" V 3045 4950 50  0000 C CNN
-F 2 "Resistor_SMD:R_1206_3216Metric_Pad1.42x1.75mm_HandSolder" H 3150 4950 50  0001 C CNN
+F 2 "Resistor_SMD:R_0805_2012Metric_Pad1.15x1.40mm_HandSolder" H 3150 4950 50  0001 C CNN
 F 3 "~" H 3150 4950 50  0001 C CNN
 	1    3150 4950
@@
 Wire Wire Line
 	8050 2800 7850 2800
+$Comp
+L Device:C C9
+U 1 1 5E1CB6EF
+P 8850 3100
+F 0 "C9" H 8965 3146 50  0000 L CNN
+F 1 "2.2uF" H 8965 3055 50  0000 L CNN
+F 2 "Capacitor_SMD:C_0805_2012Metric_Pad1.15x1.40mm_HandSolder" H 8888 2950 50  0001 C CNN
+F 3 "~" H 8850 3100 50  0001 C CNN
+	1    8850 3100
+	1    0    0    -1
+$EndComp
 $EndSCHEMATC
