File: PCB/E32CB_R2/E32CB_R2.sch (KiCad schematic (older format))
At the start: 89 parts, among them J1 GPIO_HEADER, J10 S, J11 D, J12 S, J13 D, J14 S, J15 D, J16 S, J17 D, J18 S, J19 D, J2 Power, J20 S, J21 D, J22 S, J3 USB_B, J4 USB +5V, J5 NEXTION, J6 I2C, J7 D, J8 S, J9 D, Q1 IRLR8743, Q2 IRLR8743, Q3 IRLR8743, Q4 IRLR8743, Q5 IRLR8743, Q6 IRLR8743, Q7 IRLR8743, Q8 IRLR8743, T1 S8050, T2 S8050, U1 ESP32-WROOM-32, X1 12MHz

Commit message: serial flash added
Parts:
- added J23: serial flash, Mlab_Pin_Headers:Straight_1x04, symbol MLAB_HEADER:HEADER_1x04
Connections:
- net +3V3: now also J23.1
- net GND: now also J23.4
- net RXD: now also J23.2
- net TXD: now also J23.3
Other:
- note added: "SERIAL FLASH"
Changed lines of the file:
@@
 L power:+12V #PWR017
 U 1 1 5DFA1328
-P 2400 4950
-F 0 "#PWR017" H 2400 4800 50  0001 C CNN
-F 1 "+12V" H 2415 5123 50  0000 C CNN
-F 2 "" H 2400 4950 50  0001 C CNN
-F 3 "" H 2400 4950 50  0001 C CNN
-	1    2400 4950
+P 2450 4950
+F 0 "#PWR017" H 2450 4800 50  0001 C CNN
+F 1 "+12V" H 2465 5123 50  0000 C CNN
+F 2 "" H 2450 4950 50  0001 C CNN
+F 3 "" H 2450 4950 50  0001 C CNN
+	1    2450 4950
 	-1   0    0    1
 $EndComp
@@
 Wire Wire Line
 	2250 4850 2250 4900
-Wire Wire Line
-	2350 4950 2400 4950
 Wire Wire Line
 	2250 4900 2200 4900
@@
 Text Notes 9550 1150 0    62   ~ 12
 Q7, Q8
+$Comp
+L MLAB_HEADER:HEADER_1x04 J23
+U 1 1 5F102C6A
+P 2950 5450
+F 0 "J23" V 2922 5222 60  0000 R CNN
+F 1 "serial flash" V 2816 5222 60  0000 R CNN
+F 2 "Mlab_Pin_Headers:Straight_1x04" V 2763 5222 60  0001 R CNN
+F 3 "" H 2950 5600 60  0000 C CNN
+	1    2950 5450
+	0    -1   -1   0
+$EndComp
+Wire Wire Line
+	2350 4950 2450 4950
+$Comp
+L power:+3.3V #PWR0117
+U 1 1 5F115F41
+P 2800 5950
+F 0 "#PWR0117" H 2800 5800 50  0001 C CNN
+F 1 "+3.3V" H 2815 6123 50  0000 C CNN
+F 2 "" H 2800 5950 50  0001 C CNN
+F 3 "" H 2800 5950 50  0001 C CNN
+	1    2800 5950
+	-1   0    0    1
+$EndComp
+$Comp
+L power:GND #PWR0118
+U 1 1 5F1162B7
+P 3100 5950
+F 0 "#PWR0118" H 3100 5700 50  0001 C CNN
+F 1 "GND" H 3105 5777 50  0000 C CNN
+F 2 "" H 3100 5950 50  0001 C CNN
+F 3 "" H 3100 5950 50  0001 C CNN
+	1    3100 5950
+	1    0    0    -1
+$EndComp
+Wire Wire Line
+	2800 5650 2800 5950
+Wire Wire Line
+	3100 5650 3100 5950
+Wire Wire Line
+	3000 5650 3000 5750
+Wire Wire Line
+	3000 5750 3250 5750
+Wire Wire Line
+	2900 5650 2900 5850
+Wire Wire Line
+	2900 5850 3250 5850
+Text Label 3250 5750 0    50   ~ 0
+TXD
+Text Label 3250 5850 0    50   ~ 0
+RXD
+Wire Notes Line
+	2650 5350 3750 5350
+Wire Notes Line
+	3750 5350 3750 6200
+Wire Notes Line
+	3750 6200 2650 6200
+Wire Notes Line
+	2650 6200 2650 5350
+Text Notes 2650 5350 0    50   ~ 10
+SERIAL FLASH
 $EndSCHEMATC

Commit message: schematic finished
Parts:
- removed Q1, Q2, Q3, Q4, Q5, Q6, Q7, Q8: IRLR8743, Package_TO_SOT_SMD:TO-252-2, symbol Transistor_FET:IRF8308M
- added Q1, Q2, Q3, Q4, Q5, Q6, Q7, Q8: IRLR8743, Package_TO_SOT_SMD:TO-252-2, symbol Transistor_FET:IRF740
Connections:
- net at J7.1 (Pin_1): now also Q1.2 (D)
- net at QD1.3 (D), R13.2: now also Q1.1 (G)
- net at J8.1 (Pin_1): now also Q1.3 (S)
- net at J9.1 (Pin_1): now also Q2.2 (D)
- net at QD2.3 (D), R14.2: now also Q2.1 (G)
- net at J10.1 (Pin_1): now also Q2.3 (S)
- net at J11.1 (Pin_1): now also Q3.2 (D)
- net at QD3.3 (D), R15.2: now also Q3.1 (G)
- net at J12.1 (Pin_1): now also Q3.3 (S)
- net at J13.1 (Pin_1): now also Q4.2 (D)
- net at QD4.3 (D), R16.2: now also Q4.1 (G)
- net at J14.1 (Pin_1): now also Q4.3 (S)
- net at J19.1 (Pin_1): now also Q5.2 (D)
- net at QD5.3 (D), R17.2: now also Q5.1 (G)
- net at J20.1 (Pin_1): now also Q5.3 (S)
- net at J21.1 (Pin_1): now also Q6.2 (D)
- net at QD6.3 (D), R18.2: now also Q6.1 (G)
- net at J22.1 (Pin_1): now also Q6.3 (S)
- net at J15.1 (Pin_1): now also Q7.2 (D)
- net at QD7.3 (D), R19.2: now also Q7.1 (G)
- net at J16.1 (Pin_1): now also Q7.3 (S)
- net at J17.1 (Pin_1): now also Q8.2 (D)
- net at QD8.3 (D), R20.2: now also Q8.1 (G)
- net at J18.1 (Pin_1): now also Q8.3 (S)
Changed lines of the file:
@@
-$EndComp
-$Comp
-L Transistor_FET:IRF8308M Q1
-U 1 1 5F11909A
-P 7250 4400
-F 0 "Q1" H 7455 4446 50  0000 L CNN
-F 1 "IRLR8743" H 7455 4355 50  0000 L CNN
-F 2 "Package_TO_SOT_SMD:TO-252-2" H 7250 4400 50  0001 C CIN
-F 3 "https://www.infineon.com/dgdl/irf8308mpbf.pdf?fileId=5546d462533600a40153560d319d1d61" H 7250 4400 50  0001 L CNN
-	1    7250 4400
-	1    0    0    -1
 $EndComp
 $Comp
@@
 Q1
 $Comp
-L Transistor_FET:IRF8308M Q2
-U 1 1 5F1AFF18
-P 7250 5650
-F 0 "Q2" H 7455 5696 50  0000 L CNN
-F 1 "IRLR8743" H 7455 5605 50  0000 L CNN
-F 2 "Package_TO_SOT_SMD:TO-252-2" H 7250 5650 50  0001 C CIN
-F 3 "https://www.infineon.com/dgdl/irf8308mpbf.pdf?fileId=5546d462533600a40153560d319d1d61" H 7250 5650 50  0001 L CNN
-	1    7250 5650
-	1    0    0    -1
-$EndComp
-$Comp
 L Connector_Generic:Conn_01x01 J9
 U 1 1 5F1AFF1F
@@
 Q1, Q2
 $Comp
-L Transistor_FET:IRF8308M Q3
-U 1 1 5F1E514A
-P 8850 4400
-F 0 "Q3" H 9055 4446 50  0000 L CNN
-F 1 "IRLR8743" H 9055 4355 50  0000 L CNN
-F 2 "Package_TO_SOT_SMD:TO-252-2" H 8850 4400 50  0001 C CIN
-F 3 "https://www.infineon.com/dgdl/irf8308mpbf.pdf?fileId=5546d462533600a40153560d319d1d61" H 8850 4400 50  0001 L CNN
-	1    8850 4400
-	1    0    0    -1
-$EndComp
-$Comp
 L Connector_Generic:Conn_01x01 J11
 U 1 1 5F1E5151
@@
 Q3
 $Comp
-L Transistor_FET:IRF8308M Q4
-U 1 1 5F1E5181
-P 8850 5650
-F 0 "Q4" H 9055 5696 50  0000 L CNN
-F 1 "IRLR8743" H 9055 5605 50  0000 L CNN
-F 2 "Package_TO_SOT_SMD:TO-252-2" H 8850 5650 50  0001 C CIN
-F 3 "https://www.infineon.com/dgdl/irf8308mpbf.pdf?fileId=5546d462533600a40153560d319d1d61" H 8850 5650 50  0001 L CNN
-	1    8850 5650
-	1    0    0    -1
-$EndComp
-$Comp
 L Connector_Generic:Conn_01x01 J13
 U 1 1 5F1E5188
@@
 Q3, Q4
 $Comp
-L Transistor_FET:IRF8308M Q5
-U 1 1 5F1F3ABF
-P 10450 4400
-F 0 "Q5" H 10655 4446 50  0000 L CNN
-F 1 "IRLR8743" H 10655 4355 50  0000 L CNN
-F 2 "Package_TO_SOT_SMD:TO-252-2" H 10450 4400 50  0001 C CIN
-F 3 "https://www.infineon.com/dgdl/irf8308mpbf.pdf?fileId=5546d462533600a40153560d319d1d61" H 10450 4400 50  0001 L CNN
-	1    10450 4400
-	1    0    0    -1
-$EndComp
-$Comp
 L Connector_Generic:Conn_01x01 J19
 U 1 1 5F1F3AC6
@@
 Q5
 $Comp
-L Transistor_FET:IRF8308M Q6
-U 1 1 5F1F3AF6
-P 10450 5650
-F 0 "Q6" H 10655 5696 50  0000 L CNN
-F 1 "IRLR8743" H 10655 5605 50  0000 L CNN
-F 2 "Package_TO_SOT_SMD:TO-252-2" H 10450 5650 50  0001 C CIN
-F 3 "https://www.infineon.com/dgdl/irf8308mpbf.pdf?fileId=5546d462533600a40153560d319d1d61" H 10450 5650 50  0001 L CNN
-	1    10450 5650
-	1    0    0    -1
-$EndComp
-$Comp
 L Connector_Generic:Conn_01x01 J21
 U 1 1 5F1F3AFD
@@
 Q5, Q6
 $Comp
-L Transistor_FET:IRF8308M Q7
-U 1 1 5F203D23
-P 10450 1700
-F 0 "Q7" H 10655 1746 50  0000 L CNN
-F 1 "IRLR8743" H 10655 1655 50  0000 L CNN
-F 2 "Package_TO_SOT_SMD:TO-252-2" H 10450 1700 50  0001 C CIN
-F 3 "https://www.infineon.com/dgdl/irf8308mpbf.pdf?fileId=5546d462533600a40153560d319d1d61" H 10450 1700 50  0001 L CNN
-	1    10450 1700
-	1    0    0    -1
-$EndComp
-$Comp
 L Connector_Generic:Conn_01x01 J15
 U 1 1 5F203D2A
@@
 Text Label 9600 1950 0    50   ~ 0
 Q7
-$Comp
-L Transistor_FET:IRF8308M Q8
-U 1 1 5F203D5A
-P 10450 2950
-F 0 "Q8" H 10655 2996 50  0000 L CNN
-F 1 "IRLR8743" H 10655 2905 50  0000 L CNN
-F 2 "Package_TO_SOT_SMD:TO-252-2" H 10450 2950 50  0001 C CIN
-F 3 "https://www.infineon.com/dgdl/irf8308mpbf.pdf?fileId=5546d462533600a40153560d319d1d61" H 10450 2950 50  0001 L CNN
-	1    10450 2950
-	1    0    0    -1
-$EndComp
 $Comp
 L Connector_Generic:Conn_01x01 J17
@@
 Text Notes 2650 5350 0    50   ~ 10
 SERIAL FLASH
+$Comp
+L Transistor_FET:IRF740 Q1
+U 1 1 5F1B032E
+P 7250 4400
+F 0 "Q1" H 7455 4446 50  0000 L CNN
+F 1 "IRLR8743" H 7455 4355 50  0000 L CNN
+F 2 "Package_TO_SOT_SMD:TO-252-2" H 7500 4325 50  0001 L CIN
+F 3 "http://www.vishay.com/docs/91054/91054.pdf" H 7250 4400 50  0001 L CNN
+	1    7250 4400
+	1    0    0    -1
+$EndComp
+$Comp
+L Transistor_FET:IRF740 Q2
+U 1 1 5F1FBA2A
+P 7250 5650
+F 0 "Q2" H 7455 5696 50  0000 L CNN
+F 1 "IRLR8743" H 7455 5605 50  0000 L CNN
+F 2 "Package_TO_SOT_SMD:TO-252-2" H 7500 5575 50  0001 L CIN
+F 3 "http://www.vishay.com/docs/91054/91054.pdf" H 7250 5650 50  0001 L CNN
+	1    7250 5650
+	1    0    0    -1
+$EndComp
+$Comp
+L Transistor_FET:IRF740 Q4
+U 1 1 5F1FBB5C
+P 8850 5650
+F 0 "Q4" H 9055 5696 50  0000 L CNN
+F 1 "IRLR8743" H 9055 5605 50  0000 L CNN
+F 2 "Package_TO_SOT_SMD:TO-252-2" H 9100 5575 50  0001 L CIN
+F 3 "http://www.vishay.com/docs/91054/91054.pdf" H 8850 5650 50  0001 L CNN
+	1    8850 5650
+	1    0    0    -1
+$EndComp
+$Comp
+L Transistor_FET:IRF740 Q3
+U 1 1 5F1FBC2E
+P 8850 4400
+F 0 "Q3" H 9055 4446 50  0000 L CNN
+F 1 "IRLR8743" H 9055 4355 50  0000 L CNN
+F 2 "Package_TO_SOT_SMD:TO-252-2" H 9100 4325 50  0001 L CIN
+F 3 "http://www.vishay.com/docs/91054/91054.pdf" H 8850 4400 50  0001 L CNN
+	1    8850 4400
+	1    0    0    -1
+$EndComp
+$Comp
+L Transistor_FET:IRF740 Q7
+U 1 1 5F1FBD74
+P 10450 1700
+F 0 "Q7" H 10655 1746 50  0000 L CNN
+F 1 "IRLR8743" H 10655 1655 50  0000 L CNN
+F 2 "Package_TO_SOT_SMD:TO-252-2" H 10700 1625 50  0001 L CIN
+F 3 "http://www.vishay.com/docs/91054/91054.pdf" H 10450 1700 50  0001 L CNN
+	1    10450 1700
+	1    0    0    -1
+$EndComp
+$Comp
+L Transistor_FET:IRF740 Q8
+U 1 1 5F1FBE36
+P 10450 2950
+F 0 "Q8" H 10655 2996 50  0000 L CNN
+F 1 "IRLR8743" H 10655 2905 50  0000 L CNN
+F 2 "Package_TO_SOT_SMD:TO-252-2" H 10700 2875 50  0001 L CIN
+F 3 "http://www.vishay.com/docs/91054/91054.pdf" H 10450 2950 50  0001 L CNN
+	1    10450 2950
+	1    0    0    -1
+$EndComp
+$Comp
+L Transistor_FET:IRF740 Q6
+U 1 1 5F1FBEFE
+P 10450 5650
+F 0 "Q6" H 10655 5696 50  0000 L CNN
+F 1 "IRLR8743" H 10655 5605 50  0000 L CNN
+F 2 "Package_TO_SOT_SMD:TO-252-2" H 10700 5575 50  0001 L CIN
+F 3 "http://www.vishay.com/docs/91054/91054.pdf" H 10450 5650 50  0001 L CNN
+	1    10450 5650
+	1    0    0    -1
+$EndComp
+$Comp
+L Transistor_FET:IRF740 Q5
+U 1 1 5F1FBFFC
+P 10450 4400
+F 0 "Q5" H 10655 4446 50  0000 L CNN
+F 1 "IRLR8743" H 10655 4355 50  0000 L CNN
+F 2 "Package_TO_SOT_SMD:TO-252-2" H 10700 4325 50  0001 L CIN
+F 3 "http://www.vishay.com/docs/91054/91054.pdf" H 10450 4400 50  0001 L CNN
+	1    10450 4400
+	1    0    0    -1
+$EndComp
 $EndSCHEMATC
