File: PCB/E32CB_R2/E32CB_R2.sch (KiCad schematic (older format))
At the start: 90 parts, among them J1 GPIO_HEADER, J10 S, J11 D, J12 S, J13 D, J14 S, J15 D, J16 S, J17 D, J18 S, J19 D, J2 Power, J20 S, J21 D, J22 S, J23 serial flash, J3 USB_B, J4 USB +5V, J5 NEXTION, J6 I2C, J7 D, J8 S, J9 D, Q1 IRLR8743, Q2 IRLR8743, Q3 IRLR8743, Q4 IRLR8743, Q5 IRLR8743, Q6 IRLR8743, Q7 IRLR8743, Q8 IRLR8743, T1 S8050, T2 S8050, U1 ESP32-WROOM-32, X1 12MHz

Commit message: schematics update
Parts:
- removed J1: GPIO_HEADER, Mlab_Pin_Headers:Straight_2x09, symbol MLAB_HEADER:HEADER_2x09_PARALLEL
- removed fan_1: Conn_01x04, Connector:FanPinHeader_1x04_P2.54mm_Vertical, symbol Connector_Generic:Conn_01x04
- added J1: HEADER_2x10_PARALLEL, Mlab_Pin_Headers:Straight_2x10, symbol MLAB_HEADER:HEADER_2x10_PARALLEL
- C7, C8: value 100nF -> 330nF
- C9: value 2.2uF -> 10uF
- J3: symbol Connector:USB_B -> E32CB_R2-rescue:USB_B-Connector
Connections:
- net gpi34: now also J1.11, J1.12
- net gpi35: now also J1.13, J1.14
- net gpi36: now also J1.7, J1.8
- net gpi39: now also J1.10, J1.9
- net gpio12: now also J1.17, J1.18
- net gpio15: now also J1.5, J1.6
- net gpio2: now also J1.3, J1.4
- net gpio26: now also J1.15, J1.16
- net gpio5: now also J1.1, J1.2
- net fan1 renamed gpio23
- net gpio23: now also J1.19, J1.20
Other:
- note removed: "PWM cooling fans"
- moved on the sheet: D1, J23
