File: PCB/MCPB_R1/MCPB_R1.kicad_pcb (KiCad board)
At the start: 2 copper layers, 50.3 x 9.7 mm, 10 parts, among them J1 HEADER_2x05_PARALLEL, M1 HOLE, M2 HOLE, U1 MCP9804_MSOP

Commit message: MCPB_R1 update
Parts:
- moved R1 3.79 mm to (145.0, 103.6), turned to 90 degrees
- moved A0 3.26 mm to (150.9, 101.4), turned to 90 degrees
- moved A2 2.96 mm to (154.9, 101.4), turned to 90 degrees
- moved G*** 1.42 mm to (145.3, 101.3)
- moved R2 0.90 mm to (147.3, 102.6), turned to 90 degrees
- moved J1 0.76 mm to (134.0, 101.1)
- moved A1 0.56 mm to (152.9, 101.4), turned to 90 degrees
- moved U1 0.18 mm to (153.5, 101.5), turned to 0 degrees
Routing:
- net /scl: track 19.8 -> 24.9 mm
- net /sda: track 23.1 -> 19.1 mm
- net +3V3: track 24.7 -> 27.3 mm
- net Net-(J3-Pad2): track 5.48 -> 6.92 mm
- net Net-(J2-Pad2): track 7.35 -> 8.48 mm
Other:
- board text removed: "MCPB_R1"

Commit message: MCPB update
Parts:
- removed G***: LOGO, silk_screen:logo_5mm
Changed lines of the file:
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@@
-(kicad_pcb (version 20171130) (host pcbnew 5.1.5-52549c5~84~ubuntu18.04.1)
+(kicad_pcb (version 20171130) (host pcbnew 5.0.2-bee76a0~70~ubuntu18.04.1)
   (general
     (thickness 1.6)
@@
     (tracks 52)
     (zones 0)
-    (modules 10)
+    (modules 9)
     (nets 9)
   )
@@
   )
   (setup
-    (last_trace_width 0.254)
+    (last_trace_width 0.25)
     (user_trace_width 0.254)
     (user_trace_width 0.5)
@@
     (zone_45_only no)
     (trace_min 0.2)
+    (segment_width 0.2)
+    (edge_width 0.05)
     (via_size 0.8)
     (via_drill 0.4)
@@
     (uvia_min_size 0.2)
     (uvia_min_drill 0.1)
-    (edge_width 0.05)
-    (segment_width 0.2)
     (pcb_text_width 0.3)
     (pcb_text_size 1.5 1.5)
@@
     (visible_elements FFFFFF7F)
     (pcbplotparams
-      (layerselection 0x010fc_ffffffff)
+      (layerselection 0x010f0_ffffffff)
       (usegerberextensions false)
       (usegerberattributes false)
@@
       (psa4output false)
       (plotreference true)
-      (plotvalue true)
+      (plotvalue false)
       (plotinvisibletext false)
-      (padsonsilk false)
+      (padsonsilk true)
       (subtractmaskfromsilk false)
       (outputformat 1)
@@
     (add_net "Net-(U1-Pad3)")
   )
-  (module silk_screen:logo_5mm (layer F.Cu)
-    (at 145.288 101.346 90)
-    (fp_text reference G*** (at 0 0 90) (layer F.SilkS) hide
-      (effects (font (size 1.524 1.524) (thickness 0.3)))
-    )
-    (fp_text value LOGO (at 0.75 0 90) (layer F.SilkS) hide
-      (effects (font (size 1.524 1.524) (thickness 0.3)))
-    )
-    (fp_poly (pts (xy -1.080185 -0.394483) (xy -0.994524 -0.344406) (xy -0.925098 -0.268145) (xy -0.912582 -0.247705)
-      (xy -0.875328 -0.149173) (xy -0.868367 -0.046173) (xy -0.889793 0.053607) (xy -0.937703 0.14248)
-      (xy -1.01019 0.212759) (xy -1.029777 0.225273) (xy -1.112354 0.260389) (xy -1.202743 0.277812)
-      (xy -1.285969 0.275187) (xy -1.309995 0.269304) (xy -1.410444 0.22055) (xy -1.48805 0.14931)
-      (xy -1.540444 0.061527) (xy -1.565255 -0.036853) (xy -1.560114 -0.139886) (xy -1.522649 -0.241627)
-      (xy -1.517407 -0.250865) (xy -1.451114 -0.332239) (xy -1.367543 -0.387252) (xy -1.273397 -0.415941)
-      (xy -1.175376 -0.418339) (xy -1.080185 -0.394483)) (layer F.SilkS) (width 0.01))
-    (fp_poly (pts (xy 1.320944 -1.377516) (xy 1.403486 -1.31109) (xy 1.460543 -1.22501) (xy 1.49025 -1.126487)
-      (xy 1.490747 -1.022733) (xy 1.460169 -0.92096) (xy 1.445857 -0.893924) (xy 1.385289 -0.818042)
-      (xy 1.320944 -0.768963) (xy 1.243169 -0.724437) (xy 0.071549 -0.713681) (xy 0.071549 -0.359559)
-      (xy 1.243169 -0.348803) (xy 1.320944 -0.304277) (xy 1.403242 -0.238625) (xy 1.459181 -0.155434)
-      (xy 1.488728 -0.061387) (xy 1.491853 0.036832) (xy 1.468521 0.132542) (xy 1.418702 0.219058)
-      (xy 1.342364 0.289698) (xy 1.323854 0.301367) (xy 1.243169 0.348803) (xy 0.071549 0.359559)
-      (xy 0.071549 0.642131) (xy 1.243169 0.652887) (xy 1.320944 0.697413) (xy 1.403242 0.763065)
-      (xy 1.459181 0.846256) (xy 1.488728 0.940303) (xy 1.491853 1.038522) (xy 1.468521 1.134232)
-      (xy 1.418702 1.220748) (xy 1.342364 1.291389) (xy 1.323854 1.303057) (xy 1.243169 1.350493)
-      (xy 0.456127 1.353784) (xy 0.290013 1.354138) (xy 0.13362 1.353818) (xy -0.009136 1.35288)
-      (xy -0.134341 1.351377) (xy -0.238079 1.349367) (xy -0.316434 1.346904) (xy -0.365492 1.344042)
-      (xy -0.379855 1.341983) (xy -0.481275 1.293607) (xy -0.561873 1.219689) (xy -0.590963 1.176975)
-      (xy -0.635 1.10007) (xy -0.635 -1.17162) (xy -0.587564 -1.252305) (xy -0.527074 -1.328071)
-      (xy -0.462353 -1.377516) (xy -0.384578 -1.422042) (xy 1.243169 -1.422042) (xy 1.320944 -1.377516)) (layer F.SilkS) (width 0.01))
-    (fp_poly (pts (xy 2.322634 -2.450756) (xy 2.397063 -2.391603) (xy 2.447845 -2.325545) (xy 2.495282 -2.244859)
-      (xy 2.495282 1.17162) (xy 2.447845 1.252305) (xy 2.381195 1.333967) (xy 2.297327 1.389103)
-      (xy 2.202926 1.417745) (xy 2.104674 1.419925) (xy 2.009254 1.395676) (xy 1.92335 1.345028)
-      (xy 1.853644 1.268015) (xy 1.842202 1.249395) (xy 1.797676 1.17162) (xy 1.792804 -0.308556)
-      (xy 1.787931 -1.788733) (xy -1.787932 -1.788733) (xy -1.792804 -0.308556) (xy -1.797676 1.17162)
-      (xy -1.842202 1.249395) (xy -1.903294 1.324322) (xy -1.985623 1.381319) (xy -2.079577 1.41641)
-      (xy -2.175544 1.425614) (xy -2.240136 1.414092) (xy -2.342711 1.364387) (xy -2.423268 1.28985)
-      (xy -2.451245 1.248524) (xy -2.495282 1.17162) (xy -2.495282 -2.244859) (xy -2.447846 -2.325545)
-      (xy -2.387356 -2.40131) (xy -2.322634 -2.450756) (xy -2.244859 -2.495282) (xy 2.244859 -2.495282)
-      (xy 2.322634 -2.450756)) (layer F.SilkS) (width 0.01))
-    (fp_poly (pts (xy 2.322634 1.842202) (xy 2.404615 1.907694) (xy 2.460384 1.990821) (xy 2.489941 2.084872)
-      (xy 2.493287 2.183135) (xy 2.470421 2.278899) (xy 2.421343 2.365453) (xy 2.346053 2.436085)
-      (xy 2.322634 2.450755) (xy 2.244859 2.495282) (xy 0.026831 2.498357) (xy -0.252759 2.498625)
-      (xy -0.522938 2.498654) (xy -0.781493 2.498453) (xy -1.02621 2.498034) (xy -1.254873 2.49741)
-      (xy -1.46527 2.496591) (xy -1.655185 2.495588) (xy -1.822404 2.494415) (xy -1.964713 2.493081)
-      (xy -2.079898 2.491599) (xy -2.165744 2.48998) (xy -2.220038 2.488235) (xy -2.240136 2.486555)
-      (xy -2.340825 2.438882) (xy -2.420949 2.365653) (xy -2.450724 2.321764) (xy -2.488345 2.221852)
-      (xy -2.494548 2.11789) (xy -2.471313 2.017292) (xy -2.420621 1.927471) (xy -2.344451 1.855842)
-      (xy -2.322634 1.842202) (xy -2.244859 1.797676) (xy 2.244859 1.797676) (xy 2.322634 1.842202)) (layer F.SilkS) (width 0.01))
-  )
   (module Package_SO:MSOP-8_3x3mm_P0.65mm (layer B.Cu)
